Commit message: Fix door xacro

File: cme_description/urdf/mp_model_doors.urdf.xacro (robot description, xacro)
@@ -1,19 +1,37 @@
 <?xml version="1.0"?>
-<!--
-    - Base      : kobuki
-    - Stacks    : hexagons
-    - 3d Sensor : kinect
--->
 <robot name="complete_mp_model" xmlns:xacro="http://ros.org/wiki/xacro">
-  <xacro:include filename="$(find cme_description)/urdf/mp_model.urdf.xacro" />
-  <xacro:include filename="$(find cme_description)/urdf/bim_door_v.urdf.xacro" />
-  <xacro:include filename="$(find cme_description)/urdf/bim_door_h.urdf.xacro" />
-  <!--<xacro:door_model_h name="door1" parent="building_footprint" x_loc = "10" y_loc = "10" direction_x ="1" direction_y ="0">
-  </xacro:door_model_h>-->
-  <xacro:door_model_h name="door1" parent="building_footprint" x_loc = "2.06" y_loc = "-3.5" direction_x ="1" direction_y ="0">
-  </xacro:door_model_h>
-  <xacro:door_model_v name="door2" parent="building_footprint" x_loc = "2.54" y_loc = "-4.02" direction_x ="0" direction_y ="-1">
-  </xacro:door_model_v>
-  <xacro:door_model_h name="door3" parent="building_footprint" x_loc = "3.05" y_loc = "-4.53" direction_x ="-1" direction_y ="0">
-  </xacro:door_model_h>
+	<xacro:include filename="$(find cme_description)/urdf/materials.xacro" />
+	<xacro:include filename="$(find cme_description)/urdf/mp_model.urdf.xacro" />
+	<xacro:include filename="$(find cme_description)/urdf/door.xacro.xml" />
+	<xacro:macro name="marker" params="name parent *origin">
+		<link name="${name}_marker_link">
+			<visual>
+				<geometry> <sphere radius=".1" /> </geometry>
+				<material name="red" />
+			</visual>
+		</link>
+		<joint name="${name}_marker_joint" type="fixed">
+			<xacro:insert_block name="origin" />
+			<parent link="${parent}" />
+			<child link="${name}_marker_link" />
+		</joint>
+	</xacro:macro>
+	<xacro:marker name="door1" parent="building_footprint">
+		<origin xyz="2.06 -3.5 0" rpy="0 0 0" />
+	</xacro:marker>
+	<xacro:marker name="door2" parent="building_footprint">
+		<origin xyz="2.54 -4.02 0" rpy="0 0 0"/>
+	</xacro:marker>
+	<xacro:marker name="door3" parent="building_footprint">
+		<origin xyz="3.05 -4.53 0" rpy="0 0 0"/>
+	</xacro:marker>
+	<xacro:door id="1" parent="building_footprint" width="0.70" height="2.43" depth="0.05">
+		<origin xyz="2.06 -3.5 0" rpy="0 0 0"/>
+	</xacro:door>
+	<xacro:door id="2" parent="building_footprint" width="0.70" height="2.43" depth="0.05">
+		<origin xyz="2.54 -4.02 0" rpy="0 0 ${pi/2}"/>
+	</xacro:door>
+	<xacro:door id="3" parent="building_footprint" width="0.70" height="2.43" depth="0.05">
+		<origin xyz="3.05 -4.53 0" rpy="0 0 ${pi}"/>
+	</xacro:door>
 </robot>

Commit message: More door changes, fix test world

File: cme_description/urdf/mp_model_doors.urdf.xacro (robot description, xacro)
@@ -7,5 +7,5 @@
 		<link name="${name}_marker_link">
 			<visual>
-				<geometry> <sphere radius=".1" /> </geometry>
+				<geometry> <sphere radius=".05" /> </geometry>
 				<material name="red" />
 			</visual>
@@ -17,21 +17,27 @@
 		</joint>
 	</xacro:macro>
-	<xacro:marker name="door1" parent="building_footprint">
-		<origin xyz="2.06 -3.5 0" rpy="0 0 0" />
-	</xacro:marker>
-	<xacro:marker name="door2" parent="building_footprint">
-		<origin xyz="2.54 -4.02 0" rpy="0 0 0"/>
-	</xacro:marker>
-	<xacro:marker name="door3" parent="building_footprint">
-		<origin xyz="3.05 -4.53 0" rpy="0 0 0"/>
-	</xacro:marker>
 	<xacro:door id="1" parent="building_footprint" width="0.70" height="2.43" depth="0.05">
+		<!-- origin of the door center point -->
 		<origin xyz="2.06 -3.5 0" rpy="0 0 0"/>
 	</xacro:door>
-	<xacro:door id="2" parent="building_footprint" width="0.70" height="2.43" depth="0.05">
+	<xacro:door_handle id="1" parent="door_1" door_thickness="0.05">
+		<!-- origin ${width-0.05} ${thickness/2} ${height/2}" -->
+		<origin xyz="0.65 ${0.05/2} ${2.43/2}" rpy="0 0 0"/>
+	</xacro:door_handle>
+	<xacro:door id="2" parent="building_footprint" width="0.70" height="2.43" depth="0.05" flip="true" mirror="true">
+		<!-- origin of the door center point -->
 		<origin xyz="2.54 -4.02 0" rpy="0 0 ${pi/2}"/>
 	</xacro:door>
+	<xacro:door_handle id="2" parent="door_2" door_thickness="0.05">
+		<!-- origin ${width-0.05} ${thickness/2} ${height/2}" -->
+		<origin xyz="0.65 ${0.05/2} ${2.43/2}" rpy="0 0 0"/>
+	</xacro:door_handle>
 	<xacro:door id="3" parent="building_footprint" width="0.70" height="2.43" depth="0.05">
+		<!-- origin of the door center point -->
 		<origin xyz="3.05 -4.53 0" rpy="0 0 ${pi}"/>
 	</xacro:door>
+	<xacro:door_handle id="3" parent="door_3" door_thickness="0.05">
+		<!-- origin ${width-0.05} ${thickness/2} ${height/2}" -->
+		<origin xyz="0.65 ${0.05/2} ${2.43/2}" rpy="0 0 0"/>
+	</xacro:door_handle>
 </robot>
