Commit message: xmllint --format urdf/mp_model.urdf.xacro

File: cme_description/urdf/mp_model.urdf.xacro (robot description, xacro)
@@ -1,1487 +1,1487 @@
-<?xml version = "1.0"?>
-<robot name="building" xmlns:xacro="http://www.ros.org/wiki/xacro">
-<link name = "building_footprint" ></link>
-<joint name="building_footprint_joint" type="fixed" >
-<origin xyz="0 -6 0" rpy ="0 0 0" />
-<parent link="building_footprint"/>
-<child link="floor" />
-</joint>
-<link name="floor" >
-<pose>0 0 0.1 0 0 0</pose>
-<inertial>
-<mass value="100" />
-<origin xyz="0.0 0 0" rpy =" 0 0 0" />
-<inertia ixx="10" ixy ="0"  ixz ="0" iyy = "10" iyz = "0" izz = "10" />
-</inertial>
-<visual>
-<origin xyz="0 0 0" rpy ="0 0 0" />
-<geometry name="floor_visual" >
-<box size="20 20 0.002" />
-</geometry>
-</visual>
-<collision>
-<origin xyz="0 0 0" rpy ="0 0 0" />
-<geometry name="floor_visual" >
-<box size="20 20 0.002" />
-</geometry>
-</collision>
-</link>
-<link name='Wall_0'>
-<inertial>
-<mass value="0" />
-<origin rpy="0  0  0" xyz ="0  0 1.524" />
-<inertia ixx="0" ixy ="0" ixz ="0" iyy ="0" iyz ="0" izz ="0" />
-</inertial>
-<collision name='Wall_0_Collision'>
-<origin rpy="0  0  0" xyz ="0  0 1.524" />
-<geometry>
-<box size="4.36828557853065 0.1015 3.048"/>
-</geometry>
-</collision>
-<visual name='Wall_0_Visual'>
-<origin rpy="0  0  0" xyz ="0  0 1.524" />
-<geometry>
-<box size="4.36828557853065 0.1015 3.048"/>
-</geometry>
-</visual>
-</link>
-<joint type='fixed' name='Wall_0_hinge'>
-<origin rpy="0  0 -1.5707963267949 " xyz= " -0.0320847245965127 -2.20085721073468 0" />
-<child link="Wall_0"/>
-<parent link='building_footprint'/>
-<axis xyz="0 0 0" rpy="0 0 0"/>
-<limit effort="10000" velocity="1000"/>
-<dynamics damping="1.0" friction="1.0"/>
-</joint>
-<link name='Wall_1'>
-<inertial>
-<mass value="0" />
-<origin rpy="0  0  0" xyz ="0  0 1.524" />
-<inertia ixx="0" ixy ="0" ixz ="0" iyy ="0" iyz ="0" izz ="0" />
-</inertial>
-<collision name='Wall_1_Collision'>
-<origin rpy="0  0  0" xyz ="0  0 1.524" />
-<geometry>
-<box size="5.23954304444799 0.1015 3.048"/>
-</geometry>
-</collision>
-<visual name='Wall_1_Visual'>
-<origin rpy="0  0  0" xyz ="0  0 1.524" />
-<geometry>
-<box size="5.23954304444799 0.1015 3.048"/>
-</geometry>
-</visual>
-</link>
-<joint type='fixed' name='Wall_1_hinge'>
-<origin rpy="0  0 1.5707963267949 " xyz= " -1.80696721821406 -10.1969428992453 0" />
-<child link="Wall_1"/>
-<parent link='building_footprint'/>
-<axis xyz="0 0 0" rpy="0 0 0"/>
-<limit effort="10000" velocity="1000"/>
-<dynamics damping="1.0" friction="1.0"/>
-</joint>
-<link name='Wall_2'>
-<inertial>
-<mass value="0" />
-<origin rpy="0  0  0" xyz ="0  0 1.524" />
-<inertia ixx="0" ixy ="0" ixz ="0" iyy ="0" iyz ="0" izz ="0" />
-</inertial>
-<collision name='Wall_2_Collision'>
-<origin rpy="0  0  0" xyz ="0  0 1.524" />
-<geometry>
-<box size="1.51587077327675 0.1015 3.048"/>
-</geometry>
-</collision>
-<visual name='Wall_2_Visual'>
-<origin rpy="0  0  0" xyz ="0  0 1.524" />
-<geometry>
-<box size="1.51587077327675 0.1015 3.048"/>
-</geometry>
-</visual>
-</link>
-<joint type='fixed' name='Wall_2_hinge'>
-<origin rpy="0  0 0 " xyz= " 0.765850662041855 -4.345 0" />
-<child link="Wall_2"/>
-<parent link='building_footprint'/>
-<axis xyz="0 0 0" rpy="0 0 0"/>
-<limit effort="10000" velocity="1000"/>
-<dynamics damping="1.0" friction="1.0"/>
-</joint>
-<link name='Wall_3'>
-<inertial>
-<mass value="0" />
-<origin rpy="0  0  0" xyz ="0  0 1.524" />
-<inertia ixx="0" ixy ="0" ixz ="0" iyy ="0" iyz ="0" izz ="0" />
-</inertial>
-<collision name='Wall_3_Collision'>
-<origin rpy="0  0  0" xyz ="0  0 1.524" />
-<geometry>
-<box size="4.48 0.1015 3.048"/>
-</geometry>
-</collision>
-<visual name='Wall_3_Visual'>
-<origin rpy="0  0  0" xyz ="0  0 1.524" />
-<geometry>
-<box size="4.48 0.1015 3.048"/>
-</geometry>
-</visual>
-</link>
-<joint type='fixed' name='Wall_3_hinge'>
-<origin rpy="0  0 -1.5707963267949 " xyz= " 1.56378604868023 -5.75418078207523 0" />
-<child link="Wall_3"/>
-<parent link='building_footprint'/>
-<axis xyz="0 0 0" rpy="0 0 0"/>
-<limit effort="10000" velocity="1000"/>
-<dynamics damping="1.0" friction="1.0"/>
-</joint>
-<link name='Wall_4'>
-<inertial>
-<mass value="0" />
-<origin rpy="0  0  0" xyz ="0  0 1.524" />
-<inertia ixx="0" ixy ="0" ixz ="0" iyy ="0" iyz ="0" izz ="0" />
-</inertial>
-<collision name='Wall_4_Collision'>
-<origin rpy="0  0  0" xyz ="0  0 1.524" />
-<geometry>
-<box size="0.12 0.1015 3.048"/>
-</geometry>
-</collision>
-<visual name='Wall_4_Visual'>
-<origin rpy="0  0  0" xyz ="0  0 1.524" />
-<geometry>
-<box size="0.12 0.1015 3.048"/>
-</geometry>
-</visual>
-</link>
-<joint type='fixed' name='Wall_4_hinge'>
-<origin rpy="0  0 0 " xyz= " 2.41106977281029 -3.47418078207523 0" />
-<child link="Wall_4"/>
-<parent link='building_footprint'/>
-<axis xyz="0 0 0" rpy="0 0 0"/>
-<limit effort="10000" velocity="1000"/>
-<dynamics damping="1.0" friction="1.0"/>
-</joint>
-<link name='Wall_5'>
-<inertial>
-<mass value="0" />
-<origin rpy="0  0  0" xyz ="0  0 1.524" />
-<inertia ixx="0" ixy ="0" ixz ="0" iyy ="0" iyz ="0" izz ="0" />
-</inertial>
-<collision name='Wall_5_Collision'>
-<origin rpy="0  0  0" xyz ="0  0 1.524" />
-<geometry>
-<box size="3.425 0.1015 3.048"/>
-</geometry>
-</collision>
-<visual name='Wall_5_Visual'>
-<origin rpy="0  0  0" xyz ="0  0 1.524" />
-<geometry>
-<box size="3.425 0.1015 3.048"/>
-</geometry>
-</visual>
-</link>
-<joint type='fixed' name='Wall_5_hinge'>
-<origin rpy="0  0 -1.5707963267949 " xyz= " 2.51106977281029 -1.93921442146936 0" />
-<child link="Wall_5"/>
-<parent link='building_footprint'/>
-<axis xyz="0 0 0" rpy="0 0 0"/>
-<limit effort="10000" velocity="1000"/>
-<dynamics damping="1.0" friction="1.0"/>
-</joint>
-<link name='Wall_6'>
-<inertial>
-<mass value="0" />
-<origin rpy="0  0  0" xyz ="0  0 1.524" />
-<inertia ixx="0" ixy ="0" ixz ="0" iyy ="0" iyz ="0" izz ="0" />
-</inertial>
-<collision name='Wall_6_Collision'>
-<origin rpy="0  0  0" xyz ="0  0 1.524" />
-<geometry>
-<box size="0.314999999999999 0.1015 3.048"/>
-</geometry>
-</collision>
-<visual name='Wall_6_Visual'>
-<origin rpy="0  0  0" xyz ="0  0 1.524" />
-<geometry>
-<box size="0.314999999999999 0.1015 3.048"/>
-</geometry>
-</visual>
-</link>
-<joint type='fixed' name='Wall_6_hinge'>
-<origin rpy="0  0 3.14159265358979 " xyz= " 2.47356977281029 -0.186714421469355 0" />
-<child link="Wall_6"/>
-<parent link='building_footprint'/>
-<axis xyz="0 0 0" rpy="0 0 0"/>
-<limit effort="10000" velocity="1000"/>
-<dynamics damping="1.0" friction="1.0"/>
-</joint>
-<link name='Wall_7'>
-<inertial>
-<mass value="0" />
-<origin rpy="0  0  0" xyz ="0  0 1.524" />
-<inertia ixx="0" ixy ="0" ixz ="0" iyy ="0" iyz ="0" izz ="0" />
-</inertial>
-<collision name='Wall_7_Collision'>
-<origin rpy="0  0  0" xyz ="0  0 1.524" />
-<geometry>
-<box size="0.13 0.1015 3.048"/>
-</geometry>
-</collision>
-<visual name='Wall_7_Visual'>
-<origin rpy="0  0  0" xyz ="0  0 1.524" />
-<geometry>
-<box size="0.13 0.1015 3.048"/>
-</geometry>
-</visual>
-</link>
-<joint type='fixed' name='Wall_7_hinge'>
-<origin rpy="0  0 1.5707963267949 " xyz= " 2.35606977281029 -0.081714421469355 0" />
-<child link="Wall_7"/>
-<parent link='building_footprint'/>
-<axis xyz="0 0 0" rpy="0 0 0"/>
-<limit effort="10000" velocity="1000"/>
-<dynamics damping="1.0" friction="1.0"/>
-</joint>
-<link name='Wall_8'>
-<inertial>
-<mass value="0" />
-<origin rpy="0  0  0" xyz ="0  0 1.524" />
-<inertia ixx="0" ixy ="0" ixz ="0" iyy ="0" iyz ="0" izz ="0" />
-</inertial>
-<collision name='Wall_8_Collision'>
-<origin rpy="0  0  0" xyz ="0  0 1.524" />
-<geometry>
-<box size="8.215 0.1015 3.048"/>
-</geometry>
-</collision>
-<visual name='Wall_8_Visual'>
-<origin rpy="0  0  0" xyz ="0  0 1.524" />
-<geometry>
-<box size="8.215 0.1015 3.048"/>
-</geometry>
-</visual>
-</link>
-<joint type='fixed' name='Wall_8_hinge'>
-<origin rpy="0  0 0 " xyz= " 1.20041527540349 0.0232855785306519 0" />
-<child link="Wall_8"/>
-<parent link='building_footprint'/>
-<axis xyz="0 0 0" rpy="0 0 0"/>
-<limit effort="10000" velocity="1000"/>
-<dynamics damping="1.0" friction="1.0"/>
-</joint>
-<link name='Wall_9'>
-<inertial>
-<mass value="0" />
-<origin rpy="0  0  0" xyz ="0  0 1.524" />
-<inertia ixx="0" ixy ="0" ixz ="0" iyy ="0" iyz ="0" izz ="0" />
-</inertial>
-<collision name='Wall_9_Collision'>
-<origin rpy="0  0  0" xyz ="0  0 1.524" />
-<geometry>
-<box size="12.8 0.1015 3.048"/>
-</geometry>
-</collision>
-<visual name='Wall_9_Visual'>
-<origin rpy="0  0  0" xyz ="0  0 1.524" />
-<geometry>
-<box size="12.8 0.1015 3.048"/>
-</geometry>
-</visual>
-</link>
-<joint type='fixed' name='Wall_9_hinge'>
-<origin rpy="0  0 -1.5707963267949 " xyz= " 5.26791527540349 -6.41671442146936 0" />
-<child link="Wall_9"/>
-<parent link='building_footprint'/>
-<axis xyz="0 0 0" rpy="0 0 0"/>
-<limit effort="10000" velocity="1000"/>
-<dynamics damping="1.0" friction="1.0"/>
-</joint>
-<link name='Wall_10'>
-<inertial>
-<mass value="0" />
-<origin rpy="0  0  0" xyz ="0  0 1.524" />
-<inertia ixx="0" ixy ="0" ixz ="0" iyy ="0" iyz ="0" izz ="0" />
-</inertial>
-<collision name='Wall_10_Collision'>
-<origin rpy="0  0  0" xyz ="0  0 1.524" />
-<geometry>
-<box size="7.155 0.1015 3.048"/>
-</geometry>
-</collision>
-<visual name='Wall_10_Visual'>
-<origin rpy="0  0  0" xyz ="0  0 1.524" />
-<geometry>
-<box size="7.155 0.1015 3.048"/>
-</geometry>
-</visual>
-</link>
-<joint type='fixed' name='Wall_10_hinge'>
-<origin rpy="0  0 3.14159265358979 " xyz= " 1.73041527540347 -12.8567144214694 0" />
-<child link="Wall_10"/>
-<parent link='building_footprint'/>
-<axis xyz="0 0 0" rpy="0 0 0"/>
-<limit effort="10000" velocity="1000"/>
-<dynamics damping="1.0" friction="1.0"/>
-</joint>
-<link name='Wall_11'>
-<inertial>
-<mass value="0" />
-<origin rpy="0  0  0" xyz ="0  0 1.524" />
-<inertia ixx="0" ixy ="0" ixz ="0" iyy ="0" iyz ="0" izz ="0" />
-</inertial>
-<collision name='Wall_11_Collision'>
-<origin rpy="0  0  0" xyz ="0  0 1.524" />
-<geometry>
-<box size="6.115456955552 0.1015 3.048"/>
-</geometry>
-</collision>
-<visual name='Wall_11_Visual'>
-<origin rpy="0  0  0" xyz ="0  0 1.524" />
-<geometry>
-<box size="6.115456955552 0.1015 3.048"/>
-</geometry>
-</visual>
-</link>
-<joint type='fixed' name='Wall_11_hinge'>
-<origin rpy="0  0 -1.5707963267949 " xyz= " -2.86708472459651 -3.07444289924535 0" />
-<child link="Wall_11"/>
-<parent link='building_footprint'/>
-<axis xyz="0 0 0" rpy="0 0 0"/>
-<limit effort="10000" velocity="1000"/>
-<dynamics damping="1.0" friction="1.0"/>
-</joint>
-<link name='Wall_12'>
-<inertial>
-<mass value="0" />
-<origin rpy="0  0  0" xyz ="0  0 1.524" />
-<inertia ixx="0" ixy ="0" ixz ="0" iyy ="0" iyz ="0" izz ="0" />
-</inertial>
-<collision name='Wall_12_Collision'>
-<origin rpy="0  0  0" xyz ="0  0 1.524" />
-<geometry>
-<box size="0.21 0.1015 3.048"/>
-</geometry>
-</collision>
-<visual name='Wall_12_Visual'>
-<origin rpy="0  0  0" xyz ="0  0 1.524" />
-<geometry>
-<box size="0.21 0.1015 3.048"/>
-</geometry>
-</visual>
-</link>
-<joint type='fixed' name='Wall_12_hinge'>
-<origin rpy="0  0 -1.5707963267949 " xyz= " 2.67106977281029 -0.121714421469355 0" />
-<child link="Wall_12"/>
-<parent link='building_footprint'/>
-<axis xyz="0 0 0" rpy="0 0 0"/>
-<limit effort="10000" velocity="1000"/>
-<dynamics damping="1.0" friction="1.0"/>
-</joint>
-<link name='Wall_13'>
-<inertial>
-<mass value="0" />
-<origin rpy="0  0  0" xyz ="0  0 1.524" />
-<inertia ixx="0" ixy ="0" ixz ="0" iyy ="0" iyz ="0" izz ="0" />
-</inertial>
-<collision name='Wall_13_Collision'>
-<origin rpy="0  0  0" xyz ="0  0 1.524" />
-<geometry>
-<box size="0.36 0.1015 3.048"/>
-</geometry>
-</collision>
-<visual name='Wall_13_Visual'>
-<origin rpy="0  0  0" xyz ="0  0 1.524" />
-<geometry>
-<box size="0.36 0.1015 3.048"/>
-</geometry>
-</visual>
-</link>
-<joint type='fixed' name='Wall_13_hinge'>
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