Commit message: Clean mp_model.urdf.xacro
sed -i -r 's/="\s*([0-9.-]+)\s+([0-9.-]+)\s+([0-9.-]+)\s*"/="\1 \2 \3"/g' mp_model.urdf.xacro

File: cme_description/urdf/mp_model.urdf.xacro (robot description, xacro)
@@ -11,5 +11,5 @@
     <inertial>
       <mass value="100"/>
-      <origin xyz="0.0 0 0" rpy=" 0 0 0"/>
+      <origin xyz="0.0 0 0" rpy="0 0 0"/>
       <inertia ixx="10" ixy="0" ixz="0" iyy="10" iyz="0" izz="10"/>
     </inertial>
@@ -30,9 +30,9 @@
     <inertial>
       <mass value="0"/>
-      <origin rpy="0  0  0" xyz="0  0 1.524"/>
+      <origin rpy="0 0 0" xyz="0 0 1.524"/>
       <inertia ixx="0" ixy="0" ixz="0" iyy="0" iyz="0" izz="0"/>
     </inertial>
     <collision name="Wall_0_Collision">
-      <origin rpy="0  0  0" xyz="0  0 1.524"/>
+      <origin rpy="0 0 0" xyz="0 0 1.524"/>
       <geometry>
         <box size="4.36828557853065 0.1015 3.048"/>
@@ -40,5 +40,5 @@
     </collision>
     <visual name="Wall_0_Visual">
-      <origin rpy="0  0  0" xyz="0  0 1.524"/>
+      <origin rpy="0 0 0" xyz="0 0 1.524"/>
       <geometry>
         <box size="4.36828557853065 0.1015 3.048"/>
@@ -47,5 +47,5 @@
   </link>
   <joint type="fixed" name="Wall_0_hinge">
-    <origin rpy="0  0 -1.5707963267949 " xyz=" -0.0320847245965127 -2.20085721073468 0"/>
+    <origin rpy="0 0 -1.5707963267949" xyz="-0.0320847245965127 -2.20085721073468 0"/>
     <child link="Wall_0"/>
     <parent link="building_footprint"/>
@@ -57,9 +57,9 @@
     <inertial>
       <mass value="0"/>
-      <origin rpy="0  0  0" xyz="0  0 1.524"/>
+      <origin rpy="0 0 0" xyz="0 0 1.524"/>
       <inertia ixx="0" ixy="0" ixz="0" iyy="0" iyz="0" izz="0"/>
     </inertial>
     <collision name="Wall_1_Collision">
-      <origin rpy="0  0  0" xyz="0  0 1.524"/>
+      <origin rpy="0 0 0" xyz="0 0 1.524"/>
       <geometry>
         <box size="5.23954304444799 0.1015 3.048"/>
@@ -67,5 +67,5 @@
     </collision>
     <visual name="Wall_1_Visual">
-      <origin rpy="0  0  0" xyz="0  0 1.524"/>
+      <origin rpy="0 0 0" xyz="0 0 1.524"/>
       <geometry>
         <box size="5.23954304444799 0.1015 3.048"/>
@@ -74,5 +74,5 @@
   </link>
   <joint type="fixed" name="Wall_1_hinge">
-    <origin rpy="0  0 1.5707963267949 " xyz=" -1.80696721821406 -10.1969428992453 0"/>
+    <origin rpy="0 0 1.5707963267949" xyz="-1.80696721821406 -10.1969428992453 0"/>
     <child link="Wall_1"/>
     <parent link="building_footprint"/>
@@ -84,9 +84,9 @@
     <inertial>
       <mass value="0"/>
-      <origin rpy="0  0  0" xyz="0  0 1.524"/>
+      <origin rpy="0 0 0" xyz="0 0 1.524"/>
       <inertia ixx="0" ixy="0" ixz="0" iyy="0" iyz="0" izz="0"/>
     </inertial>
     <collision name="Wall_2_Collision">
-      <origin rpy="0  0  0" xyz="0  0 1.524"/>
+      <origin rpy="0 0 0" xyz="0 0 1.524"/>
       <geometry>
         <box size="1.51587077327675 0.1015 3.048"/>
@@ -94,5 +94,5 @@
     </collision>
     <visual name="Wall_2_Visual">
-      <origin rpy="0  0  0" xyz="0  0 1.524"/>
+      <origin rpy="0 0 0" xyz="0 0 1.524"/>
       <geometry>
         <box size="1.51587077327675 0.1015 3.048"/>
@@ -101,5 +101,5 @@
   </link>
   <joint type="fixed" name="Wall_2_hinge">
-    <origin rpy="0  0 0 " xyz=" 0.765850662041855 -4.345 0"/>
+    <origin rpy="0 0 0" xyz="0.765850662041855 -4.345 0"/>
     <child link="Wall_2"/>
     <parent link="building_footprint"/>
@@ -111,9 +111,9 @@
     <inertial>
       <mass value="0"/>
-      <origin rpy="0  0  0" xyz="0  0 1.524"/>
+      <origin rpy="0 0 0" xyz="0 0 1.524"/>
       <inertia ixx="0" ixy="0" ixz="0" iyy="0" iyz="0" izz="0"/>
     </inertial>
     <collision name="Wall_3_Collision">
-      <origin rpy="0  0  0" xyz="0  0 1.524"/>
+      <origin rpy="0 0 0" xyz="0 0 1.524"/>
       <geometry>
         <box size="4.48 0.1015 3.048"/>
@@ -121,5 +121,5 @@
     </collision>
     <visual name="Wall_3_Visual">
-      <origin rpy="0  0  0" xyz="0  0 1.524"/>
+      <origin rpy="0 0 0" xyz="0 0 1.524"/>
       <geometry>
         <box size="4.48 0.1015 3.048"/>
@@ -128,5 +128,5 @@
   </link>
   <joint type="fixed" name="Wall_3_hinge">
-    <origin rpy="0  0 -1.5707963267949 " xyz=" 1.56378604868023 -5.75418078207523 0"/>
+    <origin rpy="0 0 -1.5707963267949" xyz="1.56378604868023 -5.75418078207523 0"/>
     <child link="Wall_3"/>
     <parent link="building_footprint"/>
@@ -138,9 +138,9 @@
     <inertial>
       <mass value="0"/>
-      <origin rpy="0  0  0" xyz="0  0 1.524"/>
+      <origin rpy="0 0 0" xyz="0 0 1.524"/>
       <inertia ixx="0" ixy="0" ixz="0" iyy="0" iyz="0" izz="0"/>
     </inertial>
     <collision name="Wall_4_Collision">
-      <origin rpy="0  0  0" xyz="0  0 1.524"/>
+      <origin rpy="0 0 0" xyz="0 0 1.524"/>
       <geometry>
         <box size="0.12 0.1015 3.048"/>
@@ -148,5 +148,5 @@
     </collision>
     <visual name="Wall_4_Visual">
-      <origin rpy="0  0  0" xyz="0  0 1.524"/>
+      <origin rpy="0 0 0" xyz="0 0 1.524"/>
       <geometry>
         <box size="0.12 0.1015 3.048"/>
@@ -155,5 +155,5 @@
   </link>
   <joint type="fixed" name="Wall_4_hinge">
-    <origin rpy="0  0 0 " xyz=" 2.41106977281029 -3.47418078207523 0"/>
+    <origin rpy="0 0 0" xyz="2.41106977281029 -3.47418078207523 0"/>
     <child link="Wall_4"/>
     <parent link="building_footprint"/>
@@ -165,9 +165,9 @@
     <inertial>
       <mass value="0"/>
-      <origin rpy="0  0  0" xyz="0  0 1.524"/>
+      <origin rpy="0 0 0" xyz="0 0 1.524"/>
       <inertia ixx="0" ixy="0" ixz="0" iyy="0" iyz="0" izz="0"/>
     </inertial>
     <collision name="Wall_5_Collision">
-      <origin rpy="0  0  0" xyz="0  0 1.524"/>
+      <origin rpy="0 0 0" xyz="0 0 1.524"/>
       <geometry>
         <box size="3.425 0.1015 3.048"/>
@@ -175,5 +175,5 @@
     </collision>
     <visual name="Wall_5_Visual">
-      <origin rpy="0  0  0" xyz="0  0 1.524"/>
+      <origin rpy="0 0 0" xyz="0 0 1.524"/>
       <geometry>
         <box size="3.425 0.1015 3.048"/>
@@ -182,5 +182,5 @@
   </link>
   <joint type="fixed" name="Wall_5_hinge">
-    <origin rpy="0  0 -1.5707963267949 " xyz=" 2.51106977281029 -1.93921442146936 0"/>
+    <origin rpy="0 0 -1.5707963267949" xyz="2.51106977281029 -1.93921442146936 0"/>
     <child link="Wall_5"/>
     <parent link="building_footprint"/>
@@ -192,9 +192,9 @@
     <inertial>
       <mass value="0"/>
-      <origin rpy="0  0  0" xyz="0  0 1.524"/>
+      <origin rpy="0 0 0" xyz="0 0 1.524"/>
       <inertia ixx="0" ixy="0" ixz="0" iyy="0" iyz="0" izz="0"/>
     </inertial>
     <collision name="Wall_6_Collision">
-      <origin rpy="0  0  0" xyz="0  0 1.524"/>
+      <origin rpy="0 0 0" xyz="0 0 1.524"/>
       <geometry>
         <box size="0.314999999999999 0.1015 3.048"/>
@@ -202,5 +202,5 @@
     </collision>
     <visual name="Wall_6_Visual">
-      <origin rpy="0  0  0" xyz="0  0 1.524"/>
+      <origin rpy="0 0 0" xyz="0 0 1.524"/>
       <geometry>
         <box size="0.314999999999999 0.1015 3.048"/>
@@ -209,5 +209,5 @@
   </link>
   <joint type="fixed" name="Wall_6_hinge">
-    <origin rpy="0  0 3.14159265358979 " xyz=" 2.47356977281029 -0.186714421469355 0"/>
+    <origin rpy="0 0 3.14159265358979" xyz="2.47356977281029 -0.186714421469355 0"/>
     <child link="Wall_6"/>
     <parent link="building_footprint"/>
@@ -219,9 +219,9 @@
     <inertial>
       <mass value="0"/>
-      <origin rpy="0  0  0" xyz="0  0 1.524"/>
+      <origin rpy="0 0 0" xyz="0 0 1.524"/>
       <inertia ixx="0" ixy="0" ixz="0" iyy="0" iyz="0" izz="0"/>
     </inertial>
     <collision name="Wall_7_Collision">
-      <origin rpy="0  0  0" xyz="0  0 1.524"/>
+      <origin rpy="0 0 0" xyz="0 0 1.524"/>
       <geometry>
         <box size="0.13 0.1015 3.048"/>
@@ -229,5 +229,5 @@
     </collision>
     <visual name="Wall_7_Visual">
-      <origin rpy="0  0  0" xyz="0  0 1.524"/>
+      <origin rpy="0 0 0" xyz="0 0 1.524"/>
       <geometry>
         <box size="0.13 0.1015 3.048"/>
@@ -236,5 +236,5 @@
   </link>
   <joint type="fixed" name="Wall_7_hinge">
-    <origin rpy="0  0 1.5707963267949 " xyz=" 2.35606977281029 -0.081714421469355 0"/>
+    <origin rpy="0 0 1.5707963267949" xyz="2.35606977281029 -0.081714421469355 0"/>
     <child link="Wall_7"/>
     <parent link="building_footprint"/>
@@ -246,9 +246,9 @@
     <inertial>
       <mass value="0"/>
-      <origin rpy="0  0  0" xyz="0  0 1.524"/>
+      <origin rpy="0 0 0" xyz="0 0 1.524"/>
       <inertia ixx="0" ixy="0" ixz="0" iyy="0" iyz="0" izz="0"/>
     </inertial>
     <collision name="Wall_8_Collision">
-      <origin rpy="0  0  0" xyz="0  0 1.524"/>
+      <origin rpy="0 0 0" xyz="0 0 1.524"/>
       <geometry>
         <box size="8.215 0.1015 3.048"/>
@@ -256,5 +256,5 @@
     </collision>
     <visual name="Wall_8_Visual">
-      <origin rpy="0  0  0" xyz="0  0 1.524"/>
+      <origin rpy="0 0 0" xyz="0 0 1.524"/>
       <geometry>
         <box size="8.215 0.1015 3.048"/>
@@ -263,5 +263,5 @@
   </link>
   <joint type="fixed" name="Wall_8_hinge">
-    <origin rpy="0  0 0 " xyz=" 1.20041527540349 0.0232855785306519 0"/>
+    <origin rpy="0 0 0" xyz="1.20041527540349 0.0232855785306519 0"/>
     <child link="Wall_8"/>
     <parent link="building_footprint"/>
@@ -273,9 +273,9 @@
     <inertial>
       <mass value="0"/>
-      <origin rpy="0  0  0" xyz="0  0 1.524"/>
+      <origin rpy="0 0 0" xyz="0 0 1.524"/>
       <inertia ixx="0" ixy="0" ixz="0" iyy="0" iyz="0" izz="0"/>
     </inertial>
     <collision name="Wall_9_Collision">
-      <origin rpy="0  0  0" xyz="0  0 1.524"/>
+      <origin rpy="0 0 0" xyz="0 0 1.524"/>
       <geometry>
         <box size="12.8 0.1015 3.048"/>
@@ -283,5 +283,5 @@
     </collision>
     <visual name="Wall_9_Visual">
-      <origin rpy="0  0  0" xyz="0  0 1.524"/>
+      <origin rpy="0 0 0" xyz="0 0 1.524"/>
       <geometry>
         <box size="12.8 0.1015 3.048"/>
@@ -290,5 +290,5 @@
   </link>
   <joint type="fixed" name="Wall_9_hinge">
-    <origin rpy="0  0 -1.5707963267949 " xyz=" 5.26791527540349 -6.41671442146936 0"/>
+    <origin rpy="0 0 -1.5707963267949" xyz="5.26791527540349 -6.41671442146936 0"/>
     <child link="Wall_9"/>
     <parent link="building_footprint"/>
@@ -300,9 +300,9 @@
     <inertial>
       <mass value="0"/>
-      <origin rpy="0  0  0" xyz="0  0 1.524"/>
+      <origin rpy="0 0 0" xyz="0 0 1.524"/>
       <inertia ixx="0" ixy="0" ixz="0" iyy="0" iyz="0" izz="0"/>
     </inertial>
     <collision name="Wall_10_Collision">
-      <origin rpy="0  0  0" xyz="0  0 1.524"/>
+      <origin rpy="0 0 0" xyz="0 0 1.524"/>
       <geometry>
         <box size="7.155 0.1015 3.048"/>
@@ -310,5 +310,5 @@
     </collision>
     <visual name="Wall_10_Visual">
-      <origin rpy="0  0  0" xyz="0  0 1.524"/>
+      <origin rpy="0 0 0" xyz="0 0 1.524"/>
       <geometry>
         <box size="7.155 0.1015 3.048"/>
@@ -317,5 +317,5 @@
   </link>
   <joint type="fixed" name="Wall_10_hinge">
-    <origin rpy="0  0 3.14159265358979 " xyz=" 1.73041527540347 -12.8567144214694 0"/>
+    <origin rpy="0 0 3.14159265358979" xyz="1.73041527540347 -12.8567144214694 0"/>
     <child link="Wall_10"/>
     <parent link="building_footprint"/>
@@ -327,9 +327,9 @@
     <inertial>
       <mass value="0"/>
-      <origin rpy="0  0  0" xyz="0  0 1.524"/>
+      <origin rpy="0 0 0" xyz="0 0 1.524"/>
       <inertia ixx="0" ixy="0" ixz="0" iyy="0" iyz="0" izz="0"/>
     </inertial>
     <collision name="Wall_11_Collision">
-      <origin rpy="0  0  0" xyz="0  0 1.524"/>
+      <origin rpy="0 0 0" xyz="0 0 1.524"/>
       <geometry>
         <box size="6.115456955552 0.1015 3.048"/>
@@ -337,5 +337,5 @@
     </collision>
     <visual name="Wall_11_Visual">
-      <origin rpy="0  0  0" xyz="0  0 1.524"/>
+      <origin rpy="0 0 0" xyz="0 0 1.524"/>
       <geometry>
         <box size="6.115456955552 0.1015 3.048"/>
@@ -344,5 +344,5 @@
   </link>
   <joint type="fixed" name="Wall_11_hinge">
-    <origin rpy="0  0 -1.5707963267949 " xyz=" -2.86708472459651 -3.07444289924535 0"/>
+    <origin rpy="0 0 -1.5707963267949" xyz="-2.86708472459651 -3.07444289924535 0"/>
     <child link="Wall_11"/>
     <parent link="building_footprint"/>
@@ -354,9 +354,9 @@
     <inertial>
       <mass value="0"/>
-      <origin rpy="0  0  0" xyz="0  0 1.524"/>
+      <origin rpy="0 0 0" xyz="0 0 1.524"/>
       <inertia ixx="0" ixy="0" ixz="0" iyy="0" iyz="0" izz="0"/>
     </inertial>
     <collision name="Wall_12_Collision">
-      <origin rpy="0  0  0" xyz="0  0 1.524"/>
+      <origin rpy="0 0 0" xyz="0 0 1.524"/>
       <geometry>
         <box size="0.21 0.1015 3.048"/>
@@ -364,5 +364,5 @@
     </collision>
     <visual name="Wall_12_Visual">
-      <origin rpy="0  0  0" xyz="0  0 1.524"/>
+      <origin rpy="0 0 0" xyz="0 0 1.524"/>
       <geometry>
         <box size="0.21 0.1015 3.048"/>
@@ -371,5 +371,5 @@
   </link>
   <joint type="fixed" name="Wall_12_hinge">
-    <origin rpy="0  0 -1.5707963267949 " xyz=" 2.67106977281029 -0.121714421469355 0"/>
+    <origin rpy="0 0 -1.5707963267949" xyz="2.67106977281029 -0.121714421469355 0"/>
     <child link="Wall_12"/>
     <parent link="building_footprint"/>
@@ -381,9 +381,9 @@
     <inertial>
       <mass value="0"/>
-      <origin rpy="0  0  0" xyz="0  0 1.524"/>
+      <origin rpy="0 0 0" xyz="0 0 1.524"/>
       <inertia ixx="0" ixy="0" ixz="0" iyy="0" iyz="0" izz="0"/>
     </inertial>
     <collision name="Wall_13_Collision">
-      <origin rpy="0  0  0" xyz="0  0 1.524"/>
+      <origin rpy="0 0 0" xyz="0 0 1.524"/>
       <geometry>
         <box size="0.36 0.1015 3.048"/>
@@ -391,5 +391,5 @@
     </collision>
     <visual name="Wall_13_Visual">
-      <origin rpy="0  0  0" xyz="0  0 1.524"/>
+      <origin rpy="0 0 0" xyz="0 0 1.524"/>
       <geometry>
         <box size="0.36 0.1015 3.048"/>
@@ -398,5 +398,5 @@
   </link>
   <joint type="fixed" name="Wall_13_hinge">
-    <origin rpy="0  0 3.14159265358979 " xyz=" -2.02696721821405 -7.61717137702135 0"/>
+    <origin rpy="0 0 3.14159265358979" xyz="-2.02696721821405 -7.61717137702135 0"/>
     <child link="Wall_13"/>
     <parent link="building_footprint"/>
@@ -408,9 +408,9 @@
     <inertial>
       <mass value="0"/>
-      <origin rpy="0  0  0" xyz="0  0 1.524"/>
+      <origin rpy="0 0 0" xyz="0 0 1.524"/>
       <inertia ixx="0" ixy="0" ixz="0" iyy="0" iyz="0" izz="0"/>
     </inertial>
     <collision name="Wall_14_Collision">
-      <origin rpy="0  0  0" xyz="0  0 1.524"/>
+      <origin rpy="0 0 0" xyz="0 0 1.524"/>
       <geometry>
         <box size="1.525 0.1015 3.048"/>
@@ -418,5 +418,5 @@
     </collision>
     <visual name="Wall_14_Visual">
-      <origin rpy="0  0  0" xyz="0  0 1.524"/>
+      <origin rpy="0 0 0" xyz="0 0 1.524"/>
       <geometry>
         <box size="1.525 0.1015 3.048"/>
@@ -425,5 +425,5 @@
   </link>
   <joint type="fixed" name="Wall_14_hinge">
-    <origin rpy="0  0 1.5707963267949 " xyz=" -2.16696721821405 -6.81467137702135 0"/>
+    <origin rpy="0 0 1.5707963267949" xyz="-2.16696721821405 -6.81467137702135 0"/>
     <child link="Wall_14"/>
     <parent link="building_footprint"/>
@@ -435,9 +435,9 @@
     <inertial>
       <mass value="0"/>
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
Commit message: Gazebo params

File: cme_description/urdf/mp_model.urdf.xacro (robot description, xacro)
@@ -8,5 +8,5 @@
   </joint>
   <link name="floor">
-    <pose>0 0 0.1 0 0 0</pose>
+    <origin xyz="0 0 0.1" rpy="0 0 0" />
     <inertial>
       <mass value="100"/>
