Commit message: Fix mass property
sed -i '/mass/s/value="0"/value="1"/' cme_description/urdf/mp_model.urdf.xacro

File: cme_description/urdf/mp_model.urdf.xacro (robot description, xacro)
@@ -29,5 +29,5 @@
   <link name="Wall_0">
     <inertial>
-      <mass value="0"/>
+      <mass value="1"/>
       <origin rpy="0 0 0" xyz="0 0 1.524"/>
       <inertia ixx="0" ixy="0" ixz="0" iyy="0" iyz="0" izz="0"/>
@@ -50,5 +50,4 @@
     <child link="Wall_0"/>
     <parent link="building_footprint"/>
-    <axis xyz="0 0 0" rpy="0 0 0"/>
     <limit effort="10000" velocity="1000"/>
     <dynamics damping="1.0" friction="1.0"/>
@@ -56,5 +55,5 @@
   <link name="Wall_1">
     <inertial>
-      <mass value="0"/>
+      <mass value="1"/>
       <origin rpy="0 0 0" xyz="0 0 1.524"/>
       <inertia ixx="0" ixy="0" ixz="0" iyy="0" iyz="0" izz="0"/>
@@ -77,5 +76,4 @@
     <child link="Wall_1"/>
     <parent link="building_footprint"/>
-    <axis xyz="0 0 0" rpy="0 0 0"/>
     <limit effort="10000" velocity="1000"/>
     <dynamics damping="1.0" friction="1.0"/>
@@ -83,5 +81,5 @@
   <link name="Wall_2">
     <inertial>
-      <mass value="0"/>
+      <mass value="1"/>
       <origin rpy="0 0 0" xyz="0 0 1.524"/>
       <inertia ixx="0" ixy="0" ixz="0" iyy="0" iyz="0" izz="0"/>
@@ -104,5 +102,4 @@
     <child link="Wall_2"/>
     <parent link="building_footprint"/>
-    <axis xyz="0 0 0" rpy="0 0 0"/>
     <limit effort="10000" velocity="1000"/>
     <dynamics damping="1.0" friction="1.0"/>
@@ -110,5 +107,5 @@
   <link name="Wall_3">
     <inertial>
-      <mass value="0"/>
+      <mass value="1"/>
       <origin rpy="0 0 0" xyz="0 0 1.524"/>
       <inertia ixx="0" ixy="0" ixz="0" iyy="0" iyz="0" izz="0"/>
@@ -131,5 +128,4 @@
     <child link="Wall_3"/>
     <parent link="building_footprint"/>
-    <axis xyz="0 0 0" rpy="0 0 0"/>
     <limit effort="10000" velocity="1000"/>
     <dynamics damping="1.0" friction="1.0"/>
@@ -137,5 +133,5 @@
   <link name="Wall_4">
     <inertial>
-      <mass value="0"/>
+      <mass value="1"/>
       <origin rpy="0 0 0" xyz="0 0 1.524"/>
       <inertia ixx="0" ixy="0" ixz="0" iyy="0" iyz="0" izz="0"/>
@@ -158,5 +154,4 @@
     <child link="Wall_4"/>
     <parent link="building_footprint"/>
-    <axis xyz="0 0 0" rpy="0 0 0"/>
     <limit effort="10000" velocity="1000"/>
     <dynamics damping="1.0" friction="1.0"/>
@@ -164,5 +159,5 @@
   <link name="Wall_5">
     <inertial>
-      <mass value="0"/>
+      <mass value="1"/>
       <origin rpy="0 0 0" xyz="0 0 1.524"/>
       <inertia ixx="0" ixy="0" ixz="0" iyy="0" iyz="0" izz="0"/>
@@ -185,5 +180,4 @@
     <child link="Wall_5"/>
     <parent link="building_footprint"/>
-    <axis xyz="0 0 0" rpy="0 0 0"/>
     <limit effort="10000" velocity="1000"/>
     <dynamics damping="1.0" friction="1.0"/>
@@ -191,5 +185,5 @@
   <link name="Wall_6">
     <inertial>
-      <mass value="0"/>
+      <mass value="1"/>
       <origin rpy="0 0 0" xyz="0 0 1.524"/>
       <inertia ixx="0" ixy="0" ixz="0" iyy="0" iyz="0" izz="0"/>
@@ -212,5 +206,4 @@
     <child link="Wall_6"/>
     <parent link="building_footprint"/>
-    <axis xyz="0 0 0" rpy="0 0 0"/>
     <limit effort="10000" velocity="1000"/>
     <dynamics damping="1.0" friction="1.0"/>
@@ -218,5 +211,5 @@
   <link name="Wall_7">
     <inertial>
-      <mass value="0"/>
+      <mass value="1"/>
       <origin rpy="0 0 0" xyz="0 0 1.524"/>
       <inertia ixx="0" ixy="0" ixz="0" iyy="0" iyz="0" izz="0"/>
@@ -239,5 +232,4 @@
     <child link="Wall_7"/>
     <parent link="building_footprint"/>
-    <axis xyz="0 0 0" rpy="0 0 0"/>
     <limit effort="10000" velocity="1000"/>
     <dynamics damping="1.0" friction="1.0"/>
@@ -245,5 +237,5 @@
   <link name="Wall_8">
     <inertial>
-      <mass value="0"/>
+      <mass value="1"/>
       <origin rpy="0 0 0" xyz="0 0 1.524"/>
       <inertia ixx="0" ixy="0" ixz="0" iyy="0" iyz="0" izz="0"/>
@@ -266,5 +258,4 @@
     <child link="Wall_8"/>
     <parent link="building_footprint"/>
-    <axis xyz="0 0 0" rpy="0 0 0"/>
     <limit effort="10000" velocity="1000"/>
     <dynamics damping="1.0" friction="1.0"/>
@@ -272,5 +263,5 @@
   <link name="Wall_9">
     <inertial>
-      <mass value="0"/>
+      <mass value="1"/>
       <origin rpy="0 0 0" xyz="0 0 1.524"/>
       <inertia ixx="0" ixy="0" ixz="0" iyy="0" iyz="0" izz="0"/>
@@ -293,5 +284,4 @@
     <child link="Wall_9"/>
     <parent link="building_footprint"/>
-    <axis xyz="0 0 0" rpy="0 0 0"/>
     <limit effort="10000" velocity="1000"/>
     <dynamics damping="1.0" friction="1.0"/>
@@ -299,5 +289,5 @@
   <link name="Wall_10">
     <inertial>
-      <mass value="0"/>
+      <mass value="1"/>
       <origin rpy="0 0 0" xyz="0 0 1.524"/>
       <inertia ixx="0" ixy="0" ixz="0" iyy="0" iyz="0" izz="0"/>
@@ -320,5 +310,4 @@
     <child link="Wall_10"/>
     <parent link="building_footprint"/>
-    <axis xyz="0 0 0" rpy="0 0 0"/>
     <limit effort="10000" velocity="1000"/>
     <dynamics damping="1.0" friction="1.0"/>
@@ -326,5 +315,5 @@
   <link name="Wall_11">
     <inertial>
-      <mass value="0"/>
+      <mass value="1"/>
       <origin rpy="0 0 0" xyz="0 0 1.524"/>
       <inertia ixx="0" ixy="0" ixz="0" iyy="0" iyz="0" izz="0"/>
@@ -347,5 +336,4 @@
     <child link="Wall_11"/>
     <parent link="building_footprint"/>
-    <axis xyz="0 0 0" rpy="0 0 0"/>
     <limit effort="10000" velocity="1000"/>
     <dynamics damping="1.0" friction="1.0"/>
@@ -353,5 +341,5 @@
   <link name="Wall_12">
     <inertial>
-      <mass value="0"/>
+      <mass value="1"/>
       <origin rpy="0 0 0" xyz="0 0 1.524"/>
       <inertia ixx="0" ixy="0" ixz="0" iyy="0" iyz="0" izz="0"/>
@@ -374,5 +362,4 @@
     <child link="Wall_12"/>
     <parent link="building_footprint"/>
-    <axis xyz="0 0 0" rpy="0 0 0"/>
     <limit effort="10000" velocity="1000"/>
     <dynamics damping="1.0" friction="1.0"/>
@@ -380,5 +367,5 @@
   <link name="Wall_13">
     <inertial>
-      <mass value="0"/>
+      <mass value="1"/>
       <origin rpy="0 0 0" xyz="0 0 1.524"/>
       <inertia ixx="0" ixy="0" ixz="0" iyy="0" iyz="0" izz="0"/>
@@ -401,5 +388,4 @@
     <child link="Wall_13"/>
     <parent link="building_footprint"/>
-    <axis xyz="0 0 0" rpy="0 0 0"/>
     <limit effort="10000" velocity="1000"/>
     <dynamics damping="1.0" friction="1.0"/>
@@ -407,5 +393,5 @@
   <link name="Wall_14">
     <inertial>
-      <mass value="0"/>
+      <mass value="1"/>
       <origin rpy="0 0 0" xyz="0 0 1.524"/>
       <inertia ixx="0" ixy="0" ixz="0" iyy="0" iyz="0" izz="0"/>
@@ -428,5 +414,4 @@
     <child link="Wall_14"/>
     <parent link="building_footprint"/>
-    <axis xyz="0 0 0" rpy="0 0 0"/>
     <limit effort="10000" velocity="1000"/>
     <dynamics damping="1.0" friction="1.0"/>
@@ -434,5 +419,5 @@
   <link name="Wall_15">
     <inertial>
-      <mass value="0"/>
+      <mass value="1"/>
       <origin rpy="0 0 0" xyz="0 0 1.524"/>
       <inertia ixx="0" ixy="0" ixz="0" iyy="0" iyz="0" izz="0"/>
@@ -455,5 +440,4 @@
     <child link="Wall_15"/>
     <parent link="building_footprint"/>
-    <axis xyz="0 0 0" rpy="0 0 0"/>
     <limit effort="10000" velocity="1000"/>
     <dynamics damping="1.0" friction="1.0"/>
@@ -461,5 +445,5 @@
   <link name="Wall_16">
     <inertial>
-      <mass value="0"/>
+      <mass value="1"/>
       <origin rpy="0 0 0" xyz="0 0 1.524"/>
       <inertia ixx="0" ixy="0" ixz="0" iyy="0" iyz="0" izz="0"/>
@@ -482,5 +466,4 @@
     <child link="Wall_16"/>
     <parent link="building_footprint"/>
-    <axis xyz="0 0 0" rpy="0 0 0"/>
     <limit effort="10000" velocity="1000"/>
     <dynamics damping="1.0" friction="1.0"/>
@@ -488,5 +471,5 @@
   <link name="Wall_17">
     <inertial>
-      <mass value="0"/>
+      <mass value="1"/>
       <origin rpy="0 0 0" xyz="0 0 1.524"/>
       <inertia ixx="0" ixy="0" ixz="0" iyy="0" iyz="0" izz="0"/>
@@ -509,5 +492,4 @@
     <child link="Wall_17"/>
     <parent link="building_footprint"/>
-    <axis xyz="0 0 0" rpy="0 0 0"/>
     <limit effort="10000" velocity="1000"/>
     <dynamics damping="1.0" friction="1.0"/>
@@ -515,5 +497,5 @@
   <link name="Wall_18">
     <inertial>
-      <mass value="0"/>
+      <mass value="1"/>
       <origin rpy="0 0 0" xyz="0 0 1.524"/>
       <inertia ixx="0" ixy="0" ixz="0" iyy="0" iyz="0" izz="0"/>
@@ -536,5 +518,4 @@
     <child link="Wall_18"/>
     <parent link="building_footprint"/>
-    <axis xyz="0 0 0" rpy="0 0 0"/>
     <limit effort="10000" velocity="1000"/>
     <dynamics damping="1.0" friction="1.0"/>
@@ -542,5 +523,5 @@
   <link name="Wall_19">
     <inertial>
-      <mass value="0"/>
+      <mass value="1"/>
       <origin rpy="0 0 0" xyz="0 0 1.524"/>
       <inertia ixx="0" ixy="0" ixz="0" iyy="0" iyz="0" izz="0"/>
@@ -563,5 +544,4 @@
     <child link="Wall_19"/>
     <parent link="building_footprint"/>
-    <axis xyz="0 0 0" rpy="0 0 0"/>
     <limit effort="10000" velocity="1000"/>
     <dynamics damping="1.0" friction="1.0"/>
@@ -569,5 +549,5 @@
   <link name="Wall_20">
     <inertial>
-      <mass value="0"/>
+      <mass value="1"/>
       <origin rpy="0 0 0" xyz="0 0 1.524"/>
       <inertia ixx="0" ixy="0" ixz="0" iyy="0" iyz="0" izz="0"/>
@@ -590,5 +570,4 @@
     <child link="Wall_20"/>
     <parent link="building_footprint"/>
-    <axis xyz="0 0 0" rpy="0 0 0"/>
     <limit effort="10000" velocity="1000"/>
     <dynamics damping="1.0" friction="1.0"/>
@@ -596,5 +575,5 @@
   <link name="Wall_21">
     <inertial>
-      <mass value="0"/>
+      <mass value="1"/>
       <origin rpy="0 0 0" xyz="0 0 1.524"/>
       <inertia ixx="0" ixy="0" ixz="0" iyy="0" iyz="0" izz="0"/>
@@ -617,5 +596,4 @@
     <child link="Wall_21"/>
     <parent link="building_footprint"/>
-    <axis xyz="0 0 0" rpy="0 0 0"/>
     <limit effort="10000" velocity="1000"/>
     <dynamics damping="1.0" friction="1.0"/>
@@ -623,5 +601,5 @@
   <link name="Wall_22">
     <inertial>
-      <mass value="0"/>
+      <mass value="1"/>
       <origin rpy="0 0 0" xyz="0 0 1.524"/>
       <inertia ixx="0" ixy="0" ixz="0" iyy="0" iyz="0" izz="0"/>
@@ -644,5 +622,4 @@
     <child link="Wall_22"/>
     <parent link="building_footprint"/>
-    <axis xyz="0 0 0" rpy="0 0 0"/>
     <limit effort="10000" velocity="1000"/>
     <dynamics damping="1.0" friction="1.0"/>
@@ -650,5 +627,5 @@
   <link name="Wall_23">
     <inertial>
-      <mass value="0"/>
+      <mass value="1"/>
       <origin rpy="0 0 0" xyz="0 0 1.524"/>
       <inertia ixx="0" ixy="0" ixz="0" iyy="0" iyz="0" izz="0"/>
@@ -671,5 +648,4 @@
     <child link="Wall_23"/>
     <parent link="building_footprint"/>
-    <axis xyz="0 0 0" rpy="0 0 0"/>
     <limit effort="10000" velocity="1000"/>
     <dynamics damping="1.0" friction="1.0"/>
@@ -677,5 +653,5 @@
   <link name="Wall_24">
     <inertial>
-      <mass value="0"/>
+      <mass value="1"/>
       <origin rpy="0 0 0" xyz="0 0 1.524"/>
       <inertia ixx="0" ixy="0" ixz="0" iyy="0" iyz="0" izz="0"/>
@@ -698,5 +674,4 @@
     <child link="Wall_24"/>
     <parent link="building_footprint"/>
-    <axis xyz="0 0 0" rpy="0 0 0"/>
     <limit effort="10000" velocity="1000"/>
     <dynamics damping="1.0" friction="1.0"/>
@@ -704,5 +679,5 @@
   <link name="Wall_25">
     <inertial>
-      <mass value="0"/>
+      <mass value="1"/>
       <origin rpy="0 0 0" xyz="0 0 1.524"/>
       <inertia ixx="0" ixy="0" ixz="0" iyy="0" iyz="0" izz="0"/>
@@ -725,5 +700,4 @@
     <child link="Wall_25"/>
     <parent link="building_footprint"/>
-    <axis xyz="0 0 0" rpy="0 0 0"/>
     <limit effort="10000" velocity="1000"/>
     <dynamics damping="1.0" friction="1.0"/>
@@ -731,5 +705,5 @@
   <link name="Wall_26">
     <inertial>
-      <mass value="0"/>
+      <mass value="1"/>
       <origin rpy="0 0 0" xyz="0 0 1.524"/>
       <inertia ixx="0" ixy="0" ixz="0" iyy="0" iyz="0" izz="0"/>
@@ -752,5 +726,4 @@
     <child link="Wall_26"/>
     <parent link="building_footprint"/>
-    <axis xyz="0 0 0" rpy="0 0 0"/>
     <limit effort="10000" velocity="1000"/>
     <dynamics damping="1.0" friction="1.0"/>
@@ -758,5 +731,5 @@
   <link name="Wall_27">
     <inertial>
-      <mass value="0"/>
+      <mass value="1"/>
       <origin rpy="0 0 0" xyz="0 0 1.524"/>
       <inertia ixx="0" ixy="0" ixz="0" iyy="0" iyz="0" izz="0"/>
@@ -779,5 +752,4 @@
     <child link="Wall_27"/>
     <parent link="building_footprint"/>
-    <axis xyz="0 0 0" rpy="0 0 0"/>
     <limit effort="10000" velocity="1000"/>
     <dynamics damping="1.0" friction="1.0"/>
@@ -785,5 +757,5 @@
   <link name="Wall_28">
     <inertial>
-      <mass value="0"/>
+      <mass value="1"/>
       <origin rpy="0 0 0" xyz="0 0 1.524"/>
       <inertia ixx="0" ixy="0" ixz="0" iyy="0" iyz="0" izz="0"/>
@@ -806,5 +778,4 @@
     <child link="Wall_28"/>
     <parent link="building_footprint"/>
-    <axis xyz="0 0 0" rpy="0 0 0"/>
     <limit effort="10000" velocity="1000"/>
     <dynamics damping="1.0" friction="1.0"/>
@@ -812,5 +783,5 @@
   <link name="Wall_29">
     <inertial>
-      <mass value="0"/>
+      <mass value="1"/>
       <origin rpy="0 0 0" xyz="0 0 1.524"/>
       <inertia ixx="0" ixy="0" ixz="0" iyy="0" iyz="0" izz="0"/>
@@ -833,5 +804,4 @@
     <child link="Wall_29"/>
     <parent link="building_footprint"/>
-    <axis xyz="0 0 0" rpy="0 0 0"/>
     <limit effort="10000" velocity="1000"/>
     <dynamics damping="1.0" friction="1.0"/>
@@ -839,5 +809,5 @@
   <link name="Wall_30">
     <inertial>
-      <mass value="0"/>
+      <mass value="1"/>
       <origin rpy="0 0 0" xyz="0 0 1.524"/>
       <inertia ixx="0" ixy="0" ixz="0" iyy="0" iyz="0" izz="0"/>
@@ -860,5 +830,4 @@
     <child link="Wall_30"/>
     <parent link="building_footprint"/>
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
Commit message: sync

File: cme_description/urdf/mp_model.urdf.xacro (robot description, xacro)
@@ -5,26 +5,6 @@
     <origin xyz="0 -6 0" rpy="0 0 0"/>
     <parent link="building_footprint"/>
-    <child link="floor"/>
-  </joint>
-  <link name="floor">
-    <origin xyz="0 0 0.1" rpy="0 0 0" />
-    <inertial>
-      <mass value="100"/>
-      <origin xyz="0.0 0 0" rpy="0 0 0"/>
-      <inertia ixx="10" ixy="0" ixz="0" iyy="10" iyz="0" izz="10"/>
-    </inertial>
-    <visual>
-      <origin xyz="0 0 0" rpy="0 0 0"/>
-      <geometry name="floor_visual">
-        <box size="20 20 0.002"/>
-      </geometry>
-    </visual>
-    <collision>
-      <origin xyz="0 0 0" rpy="0 0 0"/>
-      <geometry name="floor_visual">
-        <box size="20 20 0.002"/>
-      </geometry>
-    </collision>
-  </link>
+    <child link="Wall_0"/>
+  </joint>
   <link name="Wall_0">
     <inertial>
