Commit message: sync

File: cme_description/urdf/mp_model.urdf.xacro (robot description, xacro)
@@ -5,29 +5,50 @@
     <origin xyz="0 -6 0" rpy="0 0 0"/>
     <parent link="building_footprint"/>
+    <child link="floor"/>
+  </joint>
+  <link name="floor">
+    <pose>0 0 0.1 0 0 0</pose>
+    <inertial>
+      <mass value="100"/>
+      <origin xyz="0.0 0 0" rpy="0 0 0"/>
+      <inertia ixx="10" ixy="0" ixz="0" iyy="10" iyz="0" izz="10"/>
+    </inertial>
+    <visual>
+      <origin xyz="0 0 0" rpy="0 0 0"/>
+      <geometry name="floor_visual">
+        <box size="20 20 0.002"/>
+      </geometry>
+    </visual>
+    <collision>
+      <origin xyz="0 0 0" rpy="0 0 0"/>
+      <geometry name="floor_visual">
+        <box size="20 20 0.002"/>
+      </geometry>
+    </collision>
+  </link>
+  <link name="Wall_0">
+    <inertial>
+      <mass value="1"/>
+      <origin rpy="0 0 0" xyz="0 0 1.524"/>
+      <inertia ixx="0" ixy="0" ixz="0" iyy="0" iyz="0" izz="0"/>
+    </inertial>
+    <collision name="Wall_0_Collision">
+      <origin rpy="0 0 0" xyz="0 0 1.524"/>
+      <geometry>
+        <box size="4.36828557853065 0.1015 3.048"/>
+      </geometry>
+    </collision>
+    <visual name="Wall_0_Visual">
+      <origin rpy="0 0 0" xyz="0 0 1.524"/>
+      <geometry>
+        <box size="4.36828557853065 0.1015 3.048"/>
+      </geometry>
+    </visual>
+  </link>
+  <joint type="fixed" name="Wall_0_hinge">
+    <origin rpy="0 0 -1.5707963267949" xyz=" -0.0320847245965127 -2.20085721073468 0"/>
     <child link="Wall_0"/>
-  </joint>
-  <link name="Wall_0">
-    <inertial>
-      <mass value="1"/>
-      <origin rpy="0 0 0" xyz="0 0 1.524"/>
-      <inertia ixx="0" ixy="0" ixz="0" iyy="0" iyz="0" izz="0"/>
-    </inertial>
-    <collision name="Wall_0_Collision">
-      <origin rpy="0 0 0" xyz="0 0 1.524"/>
-      <geometry>
-        <box size="4.36828557853065 0.1015 3.048"/>
-      </geometry>
-    </collision>
-    <visual name="Wall_0_Visual">
-      <origin rpy="0 0 0" xyz="0 0 1.524"/>
-      <geometry>
-        <box size="4.36828557853065 0.1015 3.048"/>
-      </geometry>
-    </visual>
-  </link>
-  <joint type="fixed" name="Wall_0_hinge">
-    <origin rpy="0 0 -1.5707963267949" xyz="-0.0320847245965127 -2.20085721073468 0"/>
-    <child link="Wall_0"/>
-    <parent link="building_footprint"/>
+    <parent link="building_footprint"/>
+    <axis xyz="0 0 0" rpy="0 0 0"/>
     <limit effort="10000" velocity="1000"/>
     <dynamics damping="1.0" friction="1.0"/>
@@ -53,7 +74,8 @@
   </link>
   <joint type="fixed" name="Wall_1_hinge">
-    <origin rpy="0 0 1.5707963267949" xyz="-1.80696721821406 -10.1969428992453 0"/>
+    <origin rpy="0 0 1.5707963267949" xyz=" -1.80696721821406 -10.1969428992453 0"/>
     <child link="Wall_1"/>
     <parent link="building_footprint"/>
+    <axis xyz="0 0 0" rpy="0 0 0"/>
     <limit effort="10000" velocity="1000"/>
     <dynamics damping="1.0" friction="1.0"/>
@@ -79,7 +101,8 @@
   </link>
   <joint type="fixed" name="Wall_2_hinge">
-    <origin rpy="0 0 0" xyz="0.765850662041855 -4.345 0"/>
+    <origin rpy="0 0 0" xyz=" 0.765850662041855 -4.345 0"/>
     <child link="Wall_2"/>
     <parent link="building_footprint"/>
+    <axis xyz="0 0 0" rpy="0 0 0"/>
     <limit effort="10000" velocity="1000"/>
     <dynamics damping="1.0" friction="1.0"/>
@@ -105,7 +128,8 @@
   </link>
   <joint type="fixed" name="Wall_3_hinge">
-    <origin rpy="0 0 -1.5707963267949" xyz="1.56378604868023 -5.75418078207523 0"/>
+    <origin rpy="0 0 -1.5707963267949" xyz=" 1.56378604868023 -5.75418078207523 0"/>
     <child link="Wall_3"/>
     <parent link="building_footprint"/>
+    <axis xyz="0 0 0" rpy="0 0 0"/>
     <limit effort="10000" velocity="1000"/>
     <dynamics damping="1.0" friction="1.0"/>
@@ -131,7 +155,8 @@
   </link>
   <joint type="fixed" name="Wall_4_hinge">
-    <origin rpy="0 0 0" xyz="2.41106977281029 -3.47418078207523 0"/>
+    <origin rpy="0 0 0" xyz=" 2.41106977281029 -3.47418078207523 0"/>
     <child link="Wall_4"/>
     <parent link="building_footprint"/>
+    <axis xyz="0 0 0" rpy="0 0 0"/>
     <limit effort="10000" velocity="1000"/>
     <dynamics damping="1.0" friction="1.0"/>
@@ -157,7 +182,8 @@
   </link>
   <joint type="fixed" name="Wall_5_hinge">
-    <origin rpy="0 0 -1.5707963267949" xyz="2.51106977281029 -1.93921442146936 0"/>
+    <origin rpy="0 0 -1.5707963267949" xyz=" 2.51106977281029 -1.93921442146936 0"/>
     <child link="Wall_5"/>
     <parent link="building_footprint"/>
+    <axis xyz="0 0 0" rpy="0 0 0"/>
     <limit effort="10000" velocity="1000"/>
     <dynamics damping="1.0" friction="1.0"/>
@@ -183,7 +209,8 @@
   </link>
   <joint type="fixed" name="Wall_6_hinge">
-    <origin rpy="0 0 3.14159265358979" xyz="2.47356977281029 -0.186714421469355 0"/>
+    <origin rpy="0 0 3.14159265358979" xyz=" 2.47356977281029 -0.186714421469355 0"/>
     <child link="Wall_6"/>
     <parent link="building_footprint"/>
+    <axis xyz="0 0 0" rpy="0 0 0"/>
     <limit effort="10000" velocity="1000"/>
     <dynamics damping="1.0" friction="1.0"/>
@@ -209,7 +236,8 @@
   </link>
   <joint type="fixed" name="Wall_7_hinge">
-    <origin rpy="0 0 1.5707963267949" xyz="2.35606977281029 -0.081714421469355 0"/>
+    <origin rpy="0 0 1.5707963267949" xyz=" 2.35606977281029 -0.081714421469355 0"/>
     <child link="Wall_7"/>
     <parent link="building_footprint"/>
+    <axis xyz="0 0 0" rpy="0 0 0"/>
     <limit effort="10000" velocity="1000"/>
     <dynamics damping="1.0" friction="1.0"/>
@@ -235,7 +263,8 @@
   </link>
   <joint type="fixed" name="Wall_8_hinge">
-    <origin rpy="0 0 0" xyz="1.20041527540349 0.0232855785306519 0"/>
+    <origin rpy="0 0 0" xyz=" 1.20041527540349 0.0232855785306519 0"/>
     <child link="Wall_8"/>
     <parent link="building_footprint"/>
+    <axis xyz="0 0 0" rpy="0 0 0"/>
     <limit effort="10000" velocity="1000"/>
     <dynamics damping="1.0" friction="1.0"/>
@@ -261,7 +290,8 @@
   </link>
   <joint type="fixed" name="Wall_9_hinge">
-    <origin rpy="0 0 -1.5707963267949" xyz="5.26791527540349 -6.41671442146936 0"/>
+    <origin rpy="0 0 -1.5707963267949" xyz=" 5.26791527540349 -6.41671442146936 0"/>
     <child link="Wall_9"/>
     <parent link="building_footprint"/>
+    <axis xyz="0 0 0" rpy="0 0 0"/>
     <limit effort="10000" velocity="1000"/>
     <dynamics damping="1.0" friction="1.0"/>
@@ -287,7 +317,8 @@
   </link>
   <joint type="fixed" name="Wall_10_hinge">
-    <origin rpy="0 0 3.14159265358979" xyz="1.73041527540347 -12.8567144214694 0"/>
+    <origin rpy="0 0 3.14159265358979" xyz=" 1.73041527540347 -12.8567144214694 0"/>
     <child link="Wall_10"/>
     <parent link="building_footprint"/>
+    <axis xyz="0 0 0" rpy="0 0 0"/>
     <limit effort="10000" velocity="1000"/>
     <dynamics damping="1.0" friction="1.0"/>
@@ -313,7 +344,8 @@
   </link>
   <joint type="fixed" name="Wall_11_hinge">
-    <origin rpy="0 0 -1.5707963267949" xyz="-2.86708472459651 -3.07444289924535 0"/>
+    <origin rpy="0 0 -1.5707963267949" xyz=" -2.86708472459651 -3.07444289924535 0"/>
     <child link="Wall_11"/>
     <parent link="building_footprint"/>
+    <axis xyz="0 0 0" rpy="0 0 0"/>
     <limit effort="10000" velocity="1000"/>
     <dynamics damping="1.0" friction="1.0"/>
@@ -339,7 +371,8 @@
   </link>
   <joint type="fixed" name="Wall_12_hinge">
-    <origin rpy="0 0 -1.5707963267949" xyz="2.67106977281029 -0.121714421469355 0"/>
+    <origin rpy="0 0 -1.5707963267949" xyz=" 2.67106977281029 -0.121714421469355 0"/>
     <child link="Wall_12"/>
     <parent link="building_footprint"/>
+    <axis xyz="0 0 0" rpy="0 0 0"/>
     <limit effort="10000" velocity="1000"/>
     <dynamics damping="1.0" friction="1.0"/>
@@ -365,7 +398,8 @@
   </link>
   <joint type="fixed" name="Wall_13_hinge">
-    <origin rpy="0 0 3.14159265358979" xyz="-2.02696721821405 -7.61717137702135 0"/>
+    <origin rpy="0 0 3.14159265358979" xyz=" -2.02696721821405 -7.61717137702135 0"/>
     <child link="Wall_13"/>
     <parent link="building_footprint"/>
+    <axis xyz="0 0 0" rpy="0 0 0"/>
     <limit effort="10000" velocity="1000"/>
     <dynamics damping="1.0" friction="1.0"/>
@@ -391,7 +425,8 @@
   </link>
   <joint type="fixed" name="Wall_14_hinge">
-    <origin rpy="0 0 1.5707963267949" xyz="-2.16696721821405 -6.81467137702135 0"/>
+    <origin rpy="0 0 1.5707963267949" xyz=" -2.16696721821405 -6.81467137702135 0"/>
     <child link="Wall_14"/>
     <parent link="building_footprint"/>
+    <axis xyz="0 0 0" rpy="0 0 0"/>
     <limit effort="10000" velocity="1000"/>
     <dynamics damping="1.0" friction="1.0"/>
@@ -417,7 +452,8 @@
   </link>
   <joint type="fixed" name="Wall_15_hinge">
-    <origin rpy="0 0 3.14159265358979" xyz="-2.51702597140529 -6.09217137702135 0"/>
+    <origin rpy="0 0 3.14159265358979" xyz=" -2.51702597140529 -6.09217137702135 0"/>
     <child link="Wall_15"/>
     <parent link="building_footprint"/>
+    <axis xyz="0 0 0" rpy="0 0 0"/>
     <limit effort="10000" velocity="1000"/>
     <dynamics damping="1.0" friction="1.0"/>
@@ -443,7 +479,8 @@
   </link>
   <joint type="fixed" name="Wall_16_hinge">
-    <origin rpy="0 0 0" xyz="-1.72696721821405 -7.10717137702135 0"/>
+    <origin rpy="0 0 0" xyz=" -1.72696721821405 -7.10717137702135 0"/>
     <child link="Wall_16"/>
     <parent link="building_footprint"/>
+    <axis xyz="0 0 0" rpy="0 0 0"/>
     <limit effort="10000" velocity="1000"/>
     <dynamics damping="1.0" friction="1.0"/>
@@ -469,7 +506,8 @@
   </link>
   <joint type="fixed" name="Wall_17_hinge">
-    <origin rpy="0 0 0" xyz="0.708088522297137 -7.1081449175682 0"/>
+    <origin rpy="0 0 0" xyz=" 0.708088522297137 -7.1081449175682 0"/>
     <child link="Wall_17"/>
     <parent link="building_footprint"/>
+    <axis xyz="0 0 0" rpy="0 0 0"/>
     <limit effort="10000" velocity="1000"/>
     <dynamics damping="1.0" friction="1.0"/>
@@ -495,7 +533,8 @@
   </link>
   <joint type="fixed" name="Wall_18_hinge">
-    <origin rpy="0 0 -1.5707963267949" xyz="0.203786048680223 -7.61814491756821 0"/>
+    <origin rpy="0 0 -1.5707963267949" xyz=" 0.203786048680223 -7.61814491756821 0"/>
     <child link="Wall_18"/>
     <parent link="building_footprint"/>
+    <axis xyz="0 0 0" rpy="0 0 0"/>
     <limit effort="10000" velocity="1000"/>
     <dynamics damping="1.0" friction="1.0"/>
@@ -521,7 +560,8 @@
   </link>
   <joint type="fixed" name="Wall_19_hinge">
-    <origin rpy="0 0 3.14159265358979" xyz="0.88378604868022 -7.95418078207523 0"/>
+    <origin rpy="0 0 3.14159265358979" xyz=" 0.88378604868022 -7.95418078207523 0"/>
     <child link="Wall_19"/>
     <parent link="building_footprint"/>
+    <axis xyz="0 0 0" rpy="0 0 0"/>
     <limit effort="10000" velocity="1000"/>
     <dynamics damping="1.0" friction="1.0"/>
@@ -547,7 +587,8 @@
   </link>
   <joint type="fixed" name="Wall_20_hinge">
-    <origin rpy="0 0 -1.5707963267949" xyz="2.51257647248415 -5.82868667687965 0"/>
+    <origin rpy="0 0 -1.5707963267949" xyz=" 2.51257647248415 -5.82868667687965 0"/>
     <child link="Wall_20"/>
     <parent link="building_footprint"/>
+    <axis xyz="0 0 0" rpy="0 0 0"/>
     <limit effort="10000" velocity="1000"/>
     <dynamics damping="1.0" friction="1.0"/>
@@ -573,7 +614,8 @@
   </link>
   <joint type="fixed" name="Wall_21_hinge">
-    <origin rpy="0 0 3.14159265358979" xyz="3.89024587394381 -6.23868667687965 0"/>
+    <origin rpy="0 0 3.14159265358979" xyz=" 3.89024587394381 -6.23868667687965 0"/>
     <child link="Wall_21"/>
     <parent link="building_footprint"/>
+    <axis xyz="0 0 0" rpy="0 0 0"/>
     <limit effort="10000" velocity="1000"/>
     <dynamics damping="1.0" friction="1.0"/>
@@ -599,7 +641,8 @@
   </link>
   <joint type="fixed" name="Wall_22_hinge">
-    <origin rpy="0 0 0" xyz="2.59507647248415 -4.50368667687965 0"/>
+    <origin rpy="0 0 0" xyz=" 2.59507647248415 -4.50368667687965 0"/>
     <child link="Wall_22"/>
     <parent link="building_footprint"/>
+    <axis xyz="0 0 0" rpy="0 0 0"/>
     <limit effort="10000" velocity="1000"/>
     <dynamics damping="1.0" friction="1.0"/>
@@ -625,7 +668,8 @@
   </link>
   <joint type="fixed" name="Wall_23_hinge">
-    <origin rpy="0 0 0" xyz="4.29107807727743 -4.50455145365601 0"/>
+    <origin rpy="0 0 0" xyz=" 4.29107807727743 -4.50455145365601 0"/>
     <child link="Wall_23"/>
     <parent link="building_footprint"/>
+    <axis xyz="0 0 0" rpy="0 0 0"/>
     <limit effort="10000" velocity="1000"/>
     <dynamics damping="1.0" friction="1.0"/>
@@ -651,7 +695,8 @@
   </link>
   <joint type="fixed" name="Wall_24_hinge">
-    <origin rpy="0 0 3.14159265358979" xyz="4.33024587394381 -3.88500000000001 0"/>
+    <origin rpy="0 0 3.14159265358979" xyz=" 4.33024587394381 -3.88500000000001 0"/>
     <child link="Wall_24"/>
     <parent link="building_footprint"/>
+    <axis xyz="0 0 0" rpy="0 0 0"/>
     <limit effort="10000" velocity="1000"/>
     <dynamics damping="1.0" friction="1.0"/>
@@ -677,7 +722,8 @@
   </link>
   <joint type="fixed" name="Wall_25_hinge">
-    <origin rpy="0 0 -1.5707963267949" xyz="3.47257647248415 -4.19477572682801 0"/>
+    <origin rpy="0 0 -1.5707963267949" xyz=" 3.47257647248415 -4.19477572682801 0"/>
     <child link="Wall_25"/>
     <parent link="building_footprint"/>
+    <axis xyz="0 0 0" rpy="0 0 0"/>
     <limit effort="10000" velocity="1000"/>
     <dynamics damping="1.0" friction="1.0"/>
@@ -703,7 +749,8 @@
   </link>
   <joint type="fixed" name="Wall_26_hinge">
-    <origin rpy="0 0 0" xyz="3.89302302353287 -8.08548070884217 0"/>
+    <origin rpy="0 0 0" xyz=" 3.89302302353287 -8.08548070884217 0"/>
     <child link="Wall_26"/>
     <parent link="building_footprint"/>
+    <axis xyz="0 0 0" rpy="0 0 0"/>
     <limit effort="10000" velocity="1000"/>
     <dynamics damping="1.0" friction="1.0"/>
@@ -729,7 +776,8 @@
   </link>
   <joint type="fixed" name="Wall_27_hinge">
-    <origin rpy="0 0 -1.5707963267949" xyz="2.51813077166227 -8.02094480750642 0"/>
+    <origin rpy="0 0 -1.5707963267949" xyz=" 2.51813077166227 -8.02094480750642 0"/>
     <child link="Wall_27"/>
     <parent link="building_footprint"/>
+    <axis xyz="0 0 0" rpy="0 0 0"/>
     <limit effort="10000" velocity="1000"/>
     <dynamics damping="1.0" friction="1.0"/>
@@ -755,7 +803,8 @@
   </link>
   <joint type="fixed" name="Wall_28_hinge">
-    <origin rpy="0 0 -1.5707963267949" xyz="3.54313077166227 -8.42798070884218 0"/>
+    <origin rpy="0 0 -1.5707963267949" xyz=" 3.54313077166227 -8.42798070884218 0"/>
     <child link="Wall_28"/>
     <parent link="building_footprint"/>
+    <axis xyz="0 0 0" rpy="0 0 0"/>
     <limit effort="10000" velocity="1000"/>
     <dynamics damping="1.0" friction="1.0"/>
@@ -781,7 +830,8 @@
   </link>
   <joint type="fixed" name="Wall_29_hinge">
-    <origin rpy="0 0 0" xyz="4.40552302353287 -8.69048070884218 0"/>
+    <origin rpy="0 0 0" xyz=" 4.40552302353287 -8.69048070884218 0"/>
     <child link="Wall_29"/>
     <parent link="building_footprint"/>
+    <axis xyz="0 0 0" rpy="0 0 0"/>
     <limit effort="10000" velocity="1000"/>
     <dynamics damping="1.0" friction="1.0"/>
@@ -807,7 +857,8 @@
   </link>
   <joint type="fixed" name="Wall_30_hinge">
-    <origin rpy="0 0 -1.5707963267949" xyz="-2.73708472459651 -0.0667144214693482 0"/>
+    <origin rpy="0 0 -1.5707963267949" xyz=" -2.73708472459651 -0.0667144214693482 0"/>
     <child link="Wall_30"/>
     <parent link="building_footprint"/>
+    <axis xyz="0 0 0" rpy="0 0 0"/>
     <limit effort="10000" velocity="1000"/>
     <dynamics damping="1.0" friction="1.0"/>
@@ -833,7 +884,8 @@
   </link>
   <joint type="fixed" name="Wall_31_hinge">
-    <origin rpy="0 0 3.14159265358979" xyz="-2.76208472459651 -0.156714421469348 0"/>
+    <origin rpy="0 0 3.14159265358979" xyz=" -2.76208472459651 -0.156714421469348 0"/>
     <child link="Wall_31"/>
     <parent link="building_footprint"/>
+    <axis xyz="0 0 0" rpy="0 0 0"/>
     <limit effort="10000" velocity="1000"/>
     <dynamics damping="1.0" friction="1.0"/>
@@ -859,7 +911,8 @@
   </link>
   <joint type="fixed" name="Wall_32_hinge">
-    <origin rpy="0 0 0" xyz="-2.75708472459652 -4.035 0"/>
+    <origin rpy="0 0 0" xyz=" -2.75708472459652 -4.035 0"/>
     <child link="Wall_32"/>
     <parent link="building_footprint"/>
+    <axis xyz="0 0 0" rpy="0 0 0"/>
     <limit effort="10000" velocity="1000"/>
     <dynamics damping="1.0" friction="1.0"/>
@@ -885,7 +938,8 @@
   </link>
   <joint type="fixed" name="Wall_33_hinge">
-    <origin rpy="0 0 0" xyz="-2.75708472459652 -4.34499999999999 0"/>
+    <origin rpy="0 0 0" xyz=" -2.75708472459652 -4.34499999999999 0"/>
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
Commit message: sync

File: cme_description/urdf/mp_model.urdf.xacro (robot description, xacro)
@@ -5,26 +5,6 @@
     <origin xyz="0 -6 0" rpy="0 0 0"/>
     <parent link="building_footprint"/>
-    <child link="floor"/>
-  </joint>
-  <link name="floor">
-    <pose>0 0 0.1 0 0 0</pose>
-    <inertial>
-      <mass value="100"/>
-      <origin xyz="0.0 0 0" rpy="0 0 0"/>
-      <inertia ixx="10" ixy="0" ixz="0" iyy="10" iyz="0" izz="10"/>
-    </inertial>
-    <visual>
-      <origin xyz="0 0 0" rpy="0 0 0"/>
-      <geometry name="floor_visual">
-        <box size="20 20 0.002"/>
-      </geometry>
-    </visual>
-    <collision>
-      <origin xyz="0 0 0" rpy="0 0 0"/>
-      <geometry name="floor_visual">
-        <box size="20 20 0.002"/>
-      </geometry>
-    </collision>
-  </link>
+    <child link="Wall_0"/>
+  </joint>
   <link name="Wall_0">
     <inertial>
