Commit message: Sync

File: cme_description/urdf/building/mp_model_wider.urdf.xacro (robot description, xacro)
@@ -2,12 +2,17 @@
 <robot name="building" xmlns:xacro="http://www.ros.org/wiki/xacro">
 <link name = "building_footprint" ></link>
+<joint name="building_footprint_joint" type="fixed">
+    <origin xyz="0 0 0" rpy="0 0 0"/>
+    <parent link="world"/>
+    <child link="building_footprint"/>
+  </joint>
 <link name='Wall_0'>
 <inertial>
-<mass value="0" />
-<origin rpy="0  0  0" xyz ="0  0 1.524" />
+<mass value="1" />
+<origin rpy="0 0 0" xyz ="0 0 1.524" />
 <inertia ixx="0" ixy ="0" ixz ="0" iyy ="0" iyz ="0" izz ="0" />
 </inertial>
 <collision name='Wall_0_Collision'>
-<origin rpy="0  0  0" xyz ="0  0 1.524" />
+<origin rpy="0 0 0" xyz ="0 0 1.524" />
 <geometry>
 <box size="4.36828557853065 0.1015 3.048"/>
@@ -15,5 +20,5 @@
 </collision>
 <visual name='Wall_0_Visual'>
-<origin rpy="0  0  0" xyz ="0  0 1.524" />
+<origin rpy="0 0 0" xyz ="0 0 1.524" />
 <geometry>
 <box size="4.36828557853065 0.1015 3.048"/>
@@ -22,5 +27,5 @@
 </link>
 <joint type='fixed' name='Wall_0_hinge'>
-<origin rpy="0  0 -1.5707963267949 " xyz= " -0.032084724596503 3.79914278926532 0" />
+<origin rpy="0 0 -1.5707963267949" xyz= " -0.032084724596503 3.79914278926532 0" />
 <child link="Wall_0"/>
 <parent link='building_footprint'/>
@@ -31,10 +36,10 @@
 <link name='Wall_1'>
 <inertial>
-<mass value="0" />
-<origin rpy="0  0  0" xyz ="0  0 1.524" />
+<mass value="1" />
+<origin rpy="0 0 0" xyz ="0 0 1.524" />
 <inertia ixx="0" ixy ="0" ixz ="0" iyy ="0" iyz ="0" izz ="0" />
 </inertial>
 <collision name='Wall_1_Collision'>
-<origin rpy="0  0  0" xyz ="0  0 1.524" />
+<origin rpy="0 0 0" xyz ="0 0 1.524" />
 <geometry>
 <box size="5.23954304444798 0.1015 3.048"/>
@@ -42,5 +47,5 @@
 </collision>
 <visual name='Wall_1_Visual'>
-<origin rpy="0  0  0" xyz ="0  0 1.524" />
+<origin rpy="0 0 0" xyz ="0 0 1.524" />
 <geometry>
 <box size="5.23954304444798 0.1015 3.048"/>
@@ -49,5 +54,5 @@
 </link>
 <joint type='fixed' name='Wall_1_hinge'>
-<origin rpy="0  0 1.5707963267949 " xyz= " -1.80696721821405 -4.19694289924534 0" />
+<origin rpy="0 0 1.5707963267949" xyz= " -1.80696721821405 -4.19694289924534 0" />
 <child link="Wall_1"/>
 <parent link='building_footprint'/>
@@ -58,23 +63,23 @@
 <link name='Wall_2'>
 <inertial>
-<mass value="0" />
-<origin rpy="0  0  0" xyz ="0  0 1.524" />
+<mass value="1" />
+<origin rpy="0 0 0" xyz ="0 0 1.524" />
 <inertia ixx="0" ixy ="0" ixz ="0" iyy ="0" iyz ="0" izz ="0" />
 </inertial>
 <collision name='Wall_2_Collision'>
-<origin rpy="0  0  0" xyz ="0  0 1.524" />
-<geometry>
-<box size="1.51587077327675 0.1015 3.048"/>
+<origin rpy="0 0 0" xyz ="0 0 1.524" />
+<geometry>
+<box size="1.15587077327675 0.1015 3.048"/>
 </geometry>
 </collision>
 <visual name='Wall_2_Visual'>
-<origin rpy="0  0  0" xyz ="0  0 1.524" />
-<geometry>
-<box size="1.51587077327675 0.1015 3.048"/>
+<origin rpy="0 0 0" xyz ="0 0 1.524" />
+<geometry>
+<box size="1.15587077327675 0.1015 3.048"/>
 </geometry>
 </visual>
 </link>
 <joint type='fixed' name='Wall_2_hinge'>
-<origin rpy="0  0 0 " xyz= " 0.765850662041865 1.655 0" />
+<origin rpy="0 0 0" xyz= " 0.585850662041865 1.655 0" />
 <child link="Wall_2"/>
 <parent link='building_footprint'/>
@@ -85,23 +90,23 @@
 <link name='Wall_3'>
 <inertial>
-<mass value="0" />
-<origin rpy="0  0  0" xyz ="0  0 1.524" />
+<mass value="1" />
+<origin rpy="0 0 0" xyz ="0 0 1.524" />
 <inertia ixx="0" ixy ="0" ixz ="0" iyy ="0" iyz ="0" izz ="0" />
 </inertial>
 <collision name='Wall_3_Collision'>
-<origin rpy="0  0  0" xyz ="0  0 1.524" />
-<geometry>
-<box size="4.48 0.1015 3.048"/>
+<origin rpy="0 0 0" xyz ="0 0 1.524" />
+<geometry>
+<box size="4.26 0.1015 3.048"/>
 </geometry>
 </collision>
 <visual name='Wall_3_Visual'>
-<origin rpy="0  0  0" xyz ="0  0 1.524" />
-<geometry>
-<box size="4.48 0.1015 3.048"/>
+<origin rpy="0 0 0" xyz ="0 0 1.524" />
+<geometry>
+<box size="4.26 0.1015 3.048"/>
 </geometry>
 </visual>
 </link>
 <joint type='fixed' name='Wall_3_hinge'>
-<origin rpy="0  0 -1.5707963267949 " xyz= " 1.56378604868024 0.24581921792478 0" />
+<origin rpy="0 0 -1.5707963267949" xyz= " 1.20378604868024 0.35581921792478 0" />
 <child link="Wall_3"/>
 <parent link='building_footprint'/>
@@ -112,10 +117,10 @@
 <link name='Wall_4'>
 <inertial>
-<mass value="0" />
-<origin rpy="0  0  0" xyz ="0  0 1.524" />
+<mass value="1" />
+<origin rpy="0 0 0" xyz ="0 0 1.524" />
 <inertia ixx="0" ixy ="0" ixz ="0" iyy ="0" iyz ="0" izz ="0" />
 </inertial>
 <collision name='Wall_4_Collision'>
-<origin rpy="0  0  0" xyz ="0  0 1.524" />
+<origin rpy="0 0 0" xyz ="0 0 1.524" />
 <geometry>
 <box size="0.12 0.1015 3.048"/>
@@ -123,5 +128,5 @@
 </collision>
 <visual name='Wall_4_Visual'>
-<origin rpy="0  0  0" xyz ="0  0 1.524" />
+<origin rpy="0 0 0" xyz ="0 0 1.524" />
 <geometry>
 <box size="0.12 0.1015 3.048"/>
@@ -130,5 +135,5 @@
 </link>
 <joint type='fixed' name='Wall_4_hinge'>
-<origin rpy="0  0 0 " xyz= " 2.4110697728103 2.52581921792477 0" />
+<origin rpy="0 0 0" xyz= " 2.4710697728103 2.52581921792477 0" />
 <child link="Wall_4"/>
 <parent link='building_footprint'/>
@@ -139,10 +144,10 @@
 <link name='Wall_5'>
 <inertial>
-<mass value="0" />
-<origin rpy="0  0  0" xyz ="0  0 1.524" />
+<mass value="1" />
+<origin rpy="0 0 0" xyz ="0 0 1.524" />
 <inertia ixx="0" ixy ="0" ixz ="0" iyy ="0" iyz ="0" izz ="0" />
 </inertial>
 <collision name='Wall_5_Collision'>
-<origin rpy="0  0  0" xyz ="0  0 1.524" />
+<origin rpy="0 0 0" xyz ="0 0 1.524" />
 <geometry>
 <box size="3.425 0.1015 3.048"/>
@@ -150,5 +155,5 @@
 </collision>
 <visual name='Wall_5_Visual'>
-<origin rpy="0  0  0" xyz ="0  0 1.524" />
+<origin rpy="0 0 0" xyz ="0 0 1.524" />
 <geometry>
 <box size="3.425 0.1015 3.048"/>
@@ -157,5 +162,5 @@
 </link>
 <joint type='fixed' name='Wall_5_hinge'>
-<origin rpy="0  0 -1.5707963267949 " xyz= " 2.5110697728103 4.06078557853065 0" />
+<origin rpy="0 0 -1.5707963267949" xyz= " 2.5710697728103 4.06078557853065 0" />
 <child link="Wall_5"/>
 <parent link='building_footprint'/>
@@ -166,10 +171,10 @@
 <link name='Wall_6'>
 <inertial>
-<mass value="0" />
-<origin rpy="0  0  0" xyz ="0  0 1.524" />
+<mass value="1" />
+<origin rpy="0 0 0" xyz ="0 0 1.524" />
 <inertia ixx="0" ixy ="0" ixz ="0" iyy ="0" iyz ="0" izz ="0" />
 </inertial>
 <collision name='Wall_6_Collision'>
-<origin rpy="0  0  0" xyz ="0  0 1.524" />
+<origin rpy="0 0 0" xyz ="0 0 1.524" />
 <geometry>
 <box size="0.314999999999999 0.1015 3.048"/>
@@ -177,5 +182,5 @@
 </collision>
 <visual name='Wall_6_Visual'>
-<origin rpy="0  0  0" xyz ="0  0 1.524" />
+<origin rpy="0 0 0" xyz ="0 0 1.524" />
 <geometry>
 <box size="0.314999999999999 0.1015 3.048"/>
@@ -184,5 +189,5 @@
 </link>
 <joint type='fixed' name='Wall_6_hinge'>
-<origin rpy="0  0 3.14159265358979 " xyz= " 2.4735697728103 5.81328557853065 0" />
+<origin rpy="0 0 3.14159265358979" xyz= " 2.4735697728103 5.81328557853065 0" />
 <child link="Wall_6"/>
 <parent link='building_footprint'/>
@@ -193,10 +198,10 @@
 <link name='Wall_7'>
 <inertial>
-<mass value="0" />
-<origin rpy="0  0  0" xyz ="0  0 1.524" />
+<mass value="1" />
+<origin rpy="0 0 0" xyz ="0 0 1.524" />
 <inertia ixx="0" ixy ="0" ixz ="0" iyy ="0" iyz ="0" izz ="0" />
 </inertial>
 <collision name='Wall_7_Collision'>
-<origin rpy="0  0  0" xyz ="0  0 1.524" />
+<origin rpy="0 0 0" xyz ="0 0 1.524" />
 <geometry>
 <box size="0.129999999999999 0.1015 3.048"/>
@@ -204,5 +209,5 @@
 </collision>
 <visual name='Wall_7_Visual'>
-<origin rpy="0  0  0" xyz ="0  0 1.524" />
+<origin rpy="0 0 0" xyz ="0 0 1.524" />
 <geometry>
 <box size="0.129999999999999 0.1015 3.048"/>
@@ -211,5 +216,5 @@
 </link>
 <joint type='fixed' name='Wall_7_hinge'>
-<origin rpy="0  0 1.5707963267949 " xyz= " 2.3560697728103 5.91828557853065 0" />
+<origin rpy="0 0 1.5707963267949" xyz= " 2.3560697728103 5.91828557853065 0" />
 <child link="Wall_7"/>
 <parent link='building_footprint'/>
@@ -220,10 +225,10 @@
 <link name='Wall_8'>
 <inertial>
-<mass value="0" />
-<origin rpy="0  0  0" xyz ="0  0 1.524" />
+<mass value="1" />
+<origin rpy="0 0 0" xyz ="0 0 1.524" />
 <inertia ixx="0" ixy ="0" ixz ="0" iyy ="0" iyz ="0" izz ="0" />
 </inertial>
 <collision name='Wall_8_Collision'>
-<origin rpy="0  0  0" xyz ="0  0 1.524" />
+<origin rpy="0 0 0" xyz ="0 0 1.524" />
 <geometry>
 <box size="8.215 0.1015 3.048"/>
@@ -231,5 +236,5 @@
 </collision>
 <visual name='Wall_8_Visual'>
-<origin rpy="0  0  0" xyz ="0  0 1.524" />
+<origin rpy="0 0 0" xyz ="0 0 1.524" />
 <geometry>
 <box size="8.215 0.1015 3.048"/>
@@ -238,5 +243,5 @@
 </link>
 <joint type='fixed' name='Wall_8_hinge'>
-<origin rpy="0  0 0 " xyz= " 1.2004152754035 6.02328557853065 0" />
+<origin rpy="0 0 0" xyz= " 1.2004152754035 6.02328557853065 0" />
 <child link="Wall_8"/>
 <parent link='building_footprint'/>
@@ -247,10 +252,10 @@
 <link name='Wall_9'>
 <inertial>
-<mass value="0" />
-<origin rpy="0  0  0" xyz ="0  0 1.524" />
+<mass value="1" />
+<origin rpy="0 0 0" xyz ="0 0 1.524" />
 <inertia ixx="0" ixy ="0" ixz ="0" iyy ="0" iyz ="0" izz ="0" />
 </inertial>
 <collision name='Wall_9_Collision'>
-<origin rpy="0  0  0" xyz ="0  0 1.524" />
+<origin rpy="0 0 0" xyz ="0 0 1.524" />
 <geometry>
 <box size="12.8 0.1015 3.048"/>
@@ -258,5 +263,5 @@
 </collision>
 <visual name='Wall_9_Visual'>
-<origin rpy="0  0  0" xyz ="0  0 1.524" />
+<origin rpy="0 0 0" xyz ="0 0 1.524" />
 <geometry>
 <box size="12.8 0.1015 3.048"/>
@@ -265,5 +270,5 @@
 </link>
 <joint type='fixed' name='Wall_9_hinge'>
-<origin rpy="0  0 -1.5707963267949 " xyz= " 5.2679152754035 -0.416714421469361 0" />
+<origin rpy="0 0 -1.5707963267949" xyz= " 5.2679152754035 -0.416714421469361 0" />
 <child link="Wall_9"/>
 <parent link='building_footprint'/>
@@ -274,10 +279,10 @@
 <link name='Wall_10'>
 <inertial>
-<mass value="0" />
-<origin rpy="0  0  0" xyz ="0  0 1.524" />
+<mass value="1" />
+<origin rpy="0 0 0" xyz ="0 0 1.524" />
 <inertia ixx="0" ixy ="0" ixz ="0" iyy ="0" iyz ="0" izz ="0" />
 </inertial>
 <collision name='Wall_10_Collision'>
-<origin rpy="0  0  0" xyz ="0  0 1.524" />
+<origin rpy="0 0 0" xyz ="0 0 1.524" />
 <geometry>
 <box size="7.15488249361753 0.1015 3.048"/>
@@ -285,5 +290,5 @@
 </collision>
 <visual name='Wall_10_Visual'>
-<origin rpy="0  0  0" xyz ="0  0 1.524" />
+<origin rpy="0 0 0" xyz ="0 0 1.524" />
 <geometry>
 <box size="7.15488249361753 0.1015 3.048"/>
@@ -292,5 +297,5 @@
 </link>
 <joint type='fixed' name='Wall_10_hinge'>
-<origin rpy="0  0 3.14159265358979 " xyz= " 1.73047402859472 -6.85671442146936 0" />
+<origin rpy="0 0 3.14159265358979" xyz= " 1.73047402859472 -6.85671442146936 0" />
 <child link="Wall_10"/>
 <parent link='building_footprint'/>
@@ -301,10 +306,10 @@
 <link name='Wall_11'>
 <inertial>
-<mass value="0" />
-<origin rpy="0  0  0" xyz ="0  0 1.524" />
+<mass value="1" />
+<origin rpy="0 0 0" xyz ="0 0 1.524" />
 <inertia ixx="0" ixy ="0" ixz ="0" iyy ="0" iyz ="0" izz ="0" />
 </inertial>
 <collision name='Wall_11_Collision'>
-<origin rpy="0  0  0" xyz ="0  0 1.524" />
+<origin rpy="0 0 0" xyz ="0 0 1.524" />
 <geometry>
 <box size="6.115456955552 0.1015 3.048"/>
@@ -312,5 +317,5 @@
 </collision>
 <visual name='Wall_11_Visual'>
-<origin rpy="0  0  0" xyz ="0  0 1.524" />
+<origin rpy="0 0 0" xyz ="0 0 1.524" />
 <geometry>
 <box size="6.115456955552 0.1015 3.048"/>
@@ -319,5 +324,5 @@
 </link>
 <joint type='fixed' name='Wall_11_hinge'>
-<origin rpy="0  0 -1.5707963267949 " xyz= " -2.8670847245965 2.92555710075465 0" />
+<origin rpy="0 0 -1.5707963267949" xyz= " -2.8670847245965 2.92555710075465 0" />
 <child link="Wall_11"/>
 <parent link='building_footprint'/>
@@ -328,10 +333,10 @@
 <link name='Wall_12'>
 <inertial>
-<mass value="0" />
-<origin rpy="0  0  0" xyz ="0  0 1.524" />
+<mass value="1" />
+<origin rpy="0 0 0" xyz ="0 0 1.524" />
 <inertia ixx="0" ixy ="0" ixz ="0" iyy ="0" iyz ="0" izz ="0" />
 </inertial>
 <collision name='Wall_12_Collision'>
-<origin rpy="0  0  0" xyz ="0  0 1.524" />
+<origin rpy="0 0 0" xyz ="0 0 1.524" />
 <geometry>
 <box size="0.209999999999999 0.1015 3.048"/>
@@ -339,5 +344,5 @@
 </collision>
 <visual name='Wall_12_Visual'>
-<origin rpy="0  0  0" xyz ="0  0 1.524" />
+<origin rpy="0 0 0" xyz ="0 0 1.524" />
 <geometry>
 <box size="0.209999999999999 0.1015 3.048"/>
@@ -346,5 +351,5 @@
 </link>
 <joint type='fixed' name='Wall_12_hinge'>
-<origin rpy="0  0 -1.5707963267949 " xyz= " 2.6710697728103 5.87828557853065 0" />
+<origin rpy="0 0 -1.5707963267949" xyz= " 2.6710697728103 5.87828557853065 0" />
 <child link="Wall_12"/>
 <parent link='building_footprint'/>
@@ -355,10 +360,10 @@
 <link name='Wall_13'>
 <inertial>
-<mass value="0" />
-<origin rpy="0  0  0" xyz ="0  0 1.524" />
+<mass value="1" />
+<origin rpy="0 0 0" xyz ="0 0 1.524" />
 <inertia ixx="0" ixy ="0" ixz ="0" iyy ="0" iyz ="0" izz ="0" />
 </inertial>
 <collision name='Wall_13_Collision'>
-<origin rpy="0  0  0" xyz ="0  0 1.524" />
+<origin rpy="0 0 0" xyz ="0 0 1.524" />
 <geometry>
 <box size="0.36 0.1015 3.048"/>
@@ -366,5 +371,5 @@
 </collision>
 <visual name='Wall_13_Visual'>
-<origin rpy="0  0  0" xyz ="0  0 1.524" />
+<origin rpy="0 0 0" xyz ="0 0 1.524" />
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
File: cme_description/urdf/complete_mp_model.urdf.xacro (robot description, xacro)
@@ -5,5 +5,4 @@
 	-->
 	<xacro:arg name="world_namespace" default="/" />
-	<xacro:arg name="building" default="mp_model" />
 	<!--
 	 Includes
@@ -19,5 +18,5 @@
 	 Building
 	-->
-	<xacro:include filename="$(find cme_description)/urdf/building/$(arg building).urdf.xacro" />
+	<xacro:include filename="$(find cme_description)/urdf/building/mp_model.urdf.xacro" />
 	<!--
 	 Rooms
