Commit message: sync

File: cme_description/robots/mm_400/mm_400.urdf.xacro (robot description, xacro)
@@ -1,148 +1,171 @@
 <?xml version="1.0"?>
-<!-- Materials -->
+<!-- TODO: Add grippers for arms -->
 <robot xmlns:xacro="http://www.ros.org/wiki/xacro" name="mm_400">
-  <xacro:arg name="robot_namespace" default="/" />
-  <xacro:arg name="manipulator" default="pilz" />
-  <xacro:property name="robot_namespace" value="$(arg robot_namespace)"/>
-  <xacro:property name="manipulator" value="$(arg manipulator)"/>
-<xacro:include filename="$(find cme_description)/robots/mm_400/urdf/xacros/mp_400_gazebo.xacro" />
-<!--++++++++++++++++++++++++++++++base_link++++++++++++++++++++++++++++++++++++++++++++++++++++-->
-<!--++++++++++++++++++++body++++++++++++++++++++++++++++-->
-<xacro:include filename="$(find cme_description)/robots/mm_400/urdf/xacros/mp_400_body.xacro" />
-<!--+++++++++++++++++++castor_wheel_link++++++++++++++++++++++++-->
-<xacro:include filename="$(find cme_description)/robots/mm_400/urdf/xacros/mp_400_caster_wheel.xacro" />
-<!--+++++++++++++++++++left_wheel_link++++++++++++++++++++++++-->
-<xacro:include filename="$(find cme_description)/robots/mm_400/urdf/xacros/mp_400_fixed_wheel_left.xacro" />
-<!--+++++++++++++++++++right_wheel_link++++++++++++++++++++++++-->
-<xacro:include filename="$(find cme_description)/robots/mm_400/urdf/xacros/mp_400_fixed_wheel_right.xacro" />
-<!--+++++++++++++++++++cabinet++++++++++++++++++++++++-->
-<xacro:include filename="$(find cme_description)/robots/mm_400/urdf/xacros/cabinet.xacro" />
-<!-- PRBT -->
-<xacro:include filename="$(find cme_description)/robots/mm_400/urdf/prbt_macro.xacro" />
-<!-- Panda -->
-  <xacro:include filename="$(find cme_description)/robots/mm_400/urdf/panda_arm.xacro" />
- <!-- SENSORS -->
-<!-- SENSORS -->
-<!-- <xacro:include filename="$(find cme_description)/robots/mm_400/urdf/xacros/sick_S300.xacro" /> -->
-<!-- Microscan - Comment/Uncomment if required -->
-<xacro:include filename="$(find cme_description)/robots/mm_400/urdf/xacros/micro_scan.xacro" />
-<!-- Additional sensors if required -->
-<!-- <xacro:include filename="$(find cme_description)/robots/mm_400/urdf/xacros/imu.xacro" />
-<xacro:include filename="$(find cme_description)/robots/mm_400/urdf/xacros/ultrasonic.xacro" />
-<xacro:include filename="$(find cme_description)/robots/mm_400/urdf/xacros/camera.xacro" />-->
-  <xacro:mp_400_base name="base_link">
-  </xacro:mp_400_base>
-  <!-- Wheel Macro -->
-  <xacro:caster_wheel name="wheel_front_left" parent="base_link">
-    <origin xyz="0.165 0.155 0.036" rpy="0 0 1.57" />
-  </xacro:caster_wheel>
-  <xacro:caster_wheel name="wheel_back_left" parent="base_link">
-    <origin xyz="-0.220 0.155 0.036" rpy="0 0 1.57" />
-  </xacro:caster_wheel>
-  <xacro:caster_wheel name="wheel_front_right" parent="base_link">
-    <origin xyz="0.165 -0.155 0.036" rpy="0 0 1.57" />
-  </xacro:caster_wheel>
-   <xacro:caster_wheel name="wheel_back_right" parent="base_link">
-    <origin xyz="-0.220 -0.155 0.036" rpy="0 0 1.57" />
-  </xacro:caster_wheel>
-  <xacro:fixed_wheel_right name="fixed_wheel_right" parent="base_link">
-    <origin xyz="0. -0.26 0.074" rpy="0 0 1.57" />
-  </xacro:fixed_wheel_right>
-  <xacro:fixed_wheel_left name="fixed_wheel_left" parent="base_link">
-    <origin xyz="-0. 0.26 0.074" rpy="0 0 1.57" />
-  </xacro:fixed_wheel_left>
-  <xacro:mm_400_cabinet name="cabinet" parent="base_link">
-    <origin xyz="0.02 0 0.551" rpy="0 0 3.14" />
-  </xacro:mm_400_cabinet>
-  <!-- Robot arm -->
-  <xacro:if value="${manipulator == 'pilz'}">
-	<xacro:prbt parent="cabinet_link" prefix="pilz">
-		<origin xyz="0 0 0." rpy="0 0 0" />
-	</xacro:prbt>
-  </xacro:if>
-<!-- Panda -->
-  <xacro:if value="${manipulator == 'panda'}">
-	<xacro:panda_arm parent="base_link" prefix="panda">
-		<origin xyz="0 0 0." rpy="0 0 0" />
-	</xacro:panda_arm>
-  </xacro:if>
-  <!--+++++++++++++++++++laserscanner_link++++++++++++++++++++++++-->
-  <xacro:sick_laser_v0 name="lidar_1" parent="base_link" ros_topic="lidar_1/scan_filtered">
-    <origin xyz="0.230 0 0.110" rpy="0 3.14 3.14" />
-  </xacro:sick_laser_v0>
-       <!--+++++++++++++++++++ IMU ++++++++++++++++++++++++-->
- <!-- Comment or uncomment based on your requirement -->
-<!--   <xacro:imu name="imu_1" parent="base_link">
-    <origin xyz="0.100 0 0.300" rpy="0 0 3.14" />
-  </xacro:imu> -->
-  <!--+++++++++++++++++++ Ultra Sonic ++++++++++++++++++++++++-->
-  <!-- Comment or uncomment based on your requirement -->
-  <!-- SENSOR 1 -->
-  <!-- xacro:us_sensor name="us_1" parent="base_link">
-    <origin xyz="0.100 0 0.300" rpy="0 3.14 3.14" />
-  </xacro:us_sensor-->
-  <!-- SENSOR 2 -->
-  <!-- xacro:us_sensor name="us_2" parent="base_link">
-    <origin xyz="0.110 0 0.300" rpy="0 3.14 3.14" />
-  </xacro:us_sensor-->
-  <!-- SENSOR 3 -->
-  <!-- xacro:us_sensor name="us_3" parent="base_link">
-    <origin xyz="0.120 0 0.300" rpy="0 3.14 3.14" />
-  </xacro:us_sensor-->
-  <!-- SENSOR 4 -->
-  <!-- xacro:us_sensor name="us_4" parent="base_link">
-    <origin xyz="0.130 0 0.300" rpy="0 3.14 3.14" />
-  </xacro:us_sensor-->
-  <!-- SENSOR 5 -->
-  <!-- xacro:us_sensor name="us_5" parent="base_link">
-    <origin xyz="0.140 0 0.300" rpy="0 3.14 3.14" />
-  </xacro:us_sensor-->
-  <!-- SENSOR 6 -->
-  <!-- xacro:us_sensor name="us_6" parent="base_link">
-    <origin xyz="0.150 0 0.300" rpy="0 3.14 3.14" />
-  </xacro:us_sensor-->
-  <!-- SENSOR 7 -->
-  <!-- xacro:us_sensor name="us_7" parent="base_link">
-    <origin xyz="0.160 0 0.300" rpy="0 3.14 3.14" />
-  </xacro:us_sensor-->
-  <!-- SENSOR 8 -->
-  <!-- xacro:us_sensor name="us_8" parent="base_link">
-    <origin xyz="0.170 0 0.300" rpy="0 3.14 3.14" />
-  </xacro:us_sensor-->
-  <!-- SENSOR 9 -->
-  <!-- xacro:us_sensor name="us_9" parent="base_link">
-    <origin xyz="0.180 0 0.300" rpy="0 3.14 3.14" />
-  </xacro:us_sensor-->
-  <!-- SENSOR 10 -->
-  <!-- xacro:us_sensor name="us_10" parent="base_link">
-    <origin xyz="0.100 0 0.300" rpy="0 3.14 3.14" />
-  </xacro:us_sensor-->
-  <!-- SENSOR 11 -->
-  <!-- xacro:us_sensor name="us_11" parent="base_link">
-    <origin xyz="0.100 0 0.300" rpy="0 3.14 3.14" />
-  </xacro:us_sensor-->
-  <!-- SENSOR 12 -->
-  <!-- xacro:us_sensor name="us_12" parent="base_link">
-    <origin xyz="0.190 0 0.300" rpy="0 3.14 3.14" />
-  </xacro:us_sensor-->
-  <!-- SENSOR 13 -->
-  <!-- xacro:us_sensor name="us_13" parent="base_link">
-    <origin xyz="0.200 0 0.300" rpy="0 3.14 3.14" />
-  </xacro:us_sensor-->
-  <!-- SENSOR 14 -->
-  <!-- xacro:us_sensor name="us_14" parent="base_link">
-    <origin xyz="0.210 0 0.300" rpy="0 3.14 3.14" />
-  </xacro:us_sensor-->
-  <!-- SENSOR 15 -->
-  <!-- xacro:us_sensor name="us_15" parent="base_link">
-    <origin xyz="0.220 0 0.300" rpy="0 3.14 3.14" />
-  </xacro:us_sensor-->
-  <!-- SENSOR 16 -->
-  <!-- xacro:us_sensor name="us_16" parent="base_link">
-    <origin xyz="0.230 0 0.300" rpy="0 3.14 3.14" />
-  </xacro:us_sensor-->
-    <!--Camera  -->
-<!-- <xacro:camera name="camera" parent="base_link">
-    <origin xyz="0 0 0.38" rpy="0 0 0" />
-  </xacro:camera> -->
+	<xacro:arg name="robot_namespace" default="/" />
+	<xacro:arg name="manipulator" default="pilz" />
+	<xacro:arg name="gripper" default="true" />
+	<xacro:arg name="camera" default="false" />
+	<xacro:arg name="micro_scan" default="true" />
+	<xacro:arg name="sick_S300" default="false" />
+	<xacro:arg name="imu" default="false" />
+	<xacro:arg name="ultrasonic" default="false" />
+	<xacro:property name="robot_namespace" value="$(arg robot_namespace)"/>
+	<!--
+	 Includes
+	-->
+	<!-- mm_400 -->
+	<xacro:include filename="$(find cme_description)/robots/mm_400/urdf/xacros/mp_400_gazebo.xacro" />
+	<xacro:include filename="$(find cme_description)/robots/mm_400/urdf/xacros/mp_400_body.xacro" />
+	<xacro:include filename="$(find cme_description)/robots/mm_400/urdf/xacros/mp_400_caster_wheel.xacro" />
+	<xacro:include filename="$(find cme_description)/robots/mm_400/urdf/xacros/mp_400_wheel_left.xacro" />
+	<xacro:include filename="$(find cme_description)/robots/mm_400/urdf/xacros/mp_400_wheel_right.xacro" />
+	<xacro:include filename="$(find cme_description)/robots/mm_400/urdf/xacros/cabinet.xacro" />
+	<!-- manipulators -->
+	<xacro:if value="$(eval manipulator == 'pilz')">
+		<xacro:include filename="$(find prbt_support)/urdf/prbt_macro.xacro" />
+	</xacro:if>
+	<xacro:if value="$(eval manipulator == 'panda')">
+		<xacro:include filename="$(find franka_description)/robots/panda_arm.xacro" />
+	</xacro:if>
+	<!-- SENSORS -->
+	<xacro:if value="$(arg sick_S300)">
+		<xacro:include filename="$(find cme_description)/robots/mm_400/urdf/xacros/sick_S300.xacro" />
+	</xacro:if>
+	<xacro:if value="$(arg micro_scan)">
+		<xacro:include filename="$(find cme_description)/robots/mm_400/urdf/xacros/micro_scan.xacro" />
+	</xacro:if>
+	<xacro:if value="$(arg imu)">
+		<xacro:include filename="$(find cme_description)/robots/mm_400/urdf/xacros/imu.xacro" />
+	</xacro:if>
+	<xacro:if value="$(arg ultrasonic)">
+		<xacro:include filename="$(find cme_description)/robots/mm_400/urdf/xacros/ultrasonic.xacro" />
+	</xacro:if>
+	<xacro:if value="$(arg camera)">
+		<xacro:include filename="$(find cme_description)/robots/mm_400/urdf/xacros/camera.xacro" />
+	</xacro:if>
+	<!--
+	 Robot urdf
+	-->
+	<xacro:mp_400_base name="base_link"/>
+	<xacro:caster_wheel name="wheel_front_left" parent="base_link">
+		<origin xyz="0.165 0.155 0.036" rpy="0 0 1.57" />
+	</xacro:caster_wheel>
+	<xacro:caster_wheel name="wheel_back_left" parent="base_link">
+		<origin xyz="-0.220 0.155 0.036" rpy="0 0 1.57" />
+	</xacro:caster_wheel>
+	<xacro:caster_wheel name="wheel_front_right" parent="base_link">
+		<origin xyz="0.165 -0.155 0.036" rpy="0 0 1.57" />
+	</xacro:caster_wheel>
+	<xacro:caster_wheel name="wheel_back_right" parent="base_link">
+		<origin xyz="-0.220 -0.155 0.036" rpy="0 0 1.57" />
+	</xacro:caster_wheel>
+	<xacro:wheel name="wheel_right" parent="base_link">
+		<origin xyz="0. -0.26 0.074" rpy="0 0 1.57" />
+	</xacro:wheel>
+	<xacro:wheel name="wheel_left" parent="base_link">
+		<origin xyz="-0. 0.26 0.074" rpy="0 0 1.57" />
+	</xacro:wheel>
+	<xacro:mm_400_cabinet name="cabinet" parent="base_link">
+		<origin xyz="0.02 0 0.551" rpy="0 0 3.14" />
+	</xacro:mm_400_cabinet>
+	<!--
+	 Manipulator urdf
+	-->
+	<!-- Robot arm -->
+	<xacro:if value="${eval manipulator == 'pilz'}">
+		<xacro:prbt parent="base_link" prefix="pilz">
+			<origin xyz="0 0 0." rpy="0 0 0" />
+			<xacro:arg name="gripper" value="$(arg gripper)"/>
+		</xacro:prbt>
+	</xacro:if>
+	<!-- Panda -->
+	<xacro:if value="${eval manipulator == 'panda'}">
+		<xacro:panda_arm parent="base_link" prefix="panda">
+			<origin xyz="0 0 0." rpy="0 0 0" />
+			<xacro:arg name="gripper" value="$(arg gripper)"/>
+		</xacro:panda_arm>
+	</xacro:if>
+	<!--
+	 Sensor urdf
+	-->
+	<xacro:if value="$(arg micro_scan)">
+		<xacro:sick_laser_v0 name="lidar_1" parent="base_link" ros_topic="lidar_1/scan_filtered">
+			<origin xyz="0.230 0 0.110" rpy="0 3.14 3.14" />
+		</xacro:sick_laser_v0>
+	</xacro:if>
+	<xacro:if value="$(arg camera)">
+		<xacro:camera name="camera" parent="base_link">
+			<origin xyz="0 0 0.38" rpy="0 0 0" />
+		</xacro:camera>
+	</xacro:if>
+	<xacro:if value="$(arg imu)">
+		<xacro:imu name="imu_1" parent="base_link">
+			<origin xyz="0.100 0 0.300" rpy="0 0 3.14" />
+		</xacro:imu>
+	</xacro:if>
+	<xacro:if value="$(arg ultrasonic)">
+		<xacro:us_sensor name="us_1" parent="base_link">
+			<origin xyz="0.100 0 0.300" rpy="0 3.14 3.14" />
+		</xacro:us_sensor>
+		<!-- SENSOR 2 -->
+		<xacro:us_sensor name="us_2" parent="base_link">
+			<origin xyz="0.110 0 0.300" rpy="0 3.14 3.14" />
+		</xacro:us_sensor>
+		<!-- SENSOR 3 -->
+		<xacro:us_sensor name="us_3" parent="base_link">
+			<origin xyz="0.120 0 0.300" rpy="0 3.14 3.14" />
+		</xacro:us_sensor>
+		<!-- SENSOR 4 -->
+		<xacro:us_sensor name="us_4" parent="base_link">
+			<origin xyz="0.130 0 0.300" rpy="0 3.14 3.14" />
+		</xacro:us_sensor>
+		<!-- SENSOR 5 -->
+		<xacro:us_sensor name="us_5" parent="base_link">
+			<origin xyz="0.140 0 0.300" rpy="0 3.14 3.14" />
+		</xacro:us_sensor>
+		<!-- SENSOR 6 -->
+		<xacro:us_sensor name="us_6" parent="base_link">
+			<origin xyz="0.150 0 0.300" rpy="0 3.14 3.14" />
+		</xacro:us_sensor>
+		<!-- SENSOR 7 -->
+		<xacro:us_sensor name="us_7" parent="base_link">
+			<origin xyz="0.160 0 0.300" rpy="0 3.14 3.14" />
+		</xacro:us_sensor>
+		<!-- SENSOR 8 -->
+		<xacro:us_sensor name="us_8" parent="base_link">
+			<origin xyz="0.170 0 0.300" rpy="0 3.14 3.14" />
+		</xacro:us_sensor>
+		<!-- SENSOR 9 -->
+		<xacro:us_sensor name="us_9" parent="base_link">
+			<origin xyz="0.180 0 0.300" rpy="0 3.14 3.14" />
+		</xacro:us_sensor>
+		<!-- SENSOR 10 -->
+		<xacro:us_sensor name="us_10" parent="base_link">
+			<origin xyz="0.100 0 0.300" rpy="0 3.14 3.14" />
+		</xacro:us_sensor>
+		<!-- SENSOR 11 -->
+		<xacro:us_sensor name="us_11" parent="base_link">
+			<origin xyz="0.100 0 0.300" rpy="0 3.14 3.14" />
+		</xacro:us_sensor>
+		<!-- SENSOR 12 -->
+		<xacro:us_sensor name="us_12" parent="base_link">
+			<origin xyz="0.190 0 0.300" rpy="0 3.14 3.14" />
+		</xacro:us_sensor>
+		<!-- SENSOR 13 -->
+		<xacro:us_sensor name="us_13" parent="base_link">
+			<origin xyz="0.200 0 0.300" rpy="0 3.14 3.14" />
+		</xacro:us_sensor>
+		<!-- SENSOR 14 -->
+		<xacro:us_sensor name="us_14" parent="base_link">
+			<origin xyz="0.210 0 0.300" rpy="0 3.14 3.14" />
+		</xacro:us_sensor>
+		<!-- SENSOR 15 -->
+		<xacro:us_sensor name="us_15" parent="base_link">
+			<origin xyz="0.220 0 0.300" rpy="0 3.14 3.14" />
+		</xacro:us_sensor>
+		<!-- SENSOR 16 -->
+		<xacro:us_sensor name="us_16" parent="base_link">
+			<origin xyz="0.230 0 0.300" rpy="0 3.14 3.14" />
+		</xacro:us_sensor>
+	</xacro:if>
 </robot>

File: cme_description/robots/mm_400/urdf/xacros/mp_400_caster_wheel.xacro (robot description, xacro)
@@ -5,5 +5,5 @@
     <xacro:insert_block name="origin" />
     <axis xyz="-1 0 0" />
-    <joint_properties damping="1." friction="1.0" />
+    <joint_properties damping="1" friction="1" />
     <limit effort="1000.0" lower="-1e+16" upper="1e+16" velocity="3.5"/>
     <parent link="${parent}" />
@@ -31,12 +31,10 @@
     </link>
 <gazebo reference="${name}_link">
-      <kp>10000.0</kp>
-      <kd>10.0</kd>
-      <mu1>0.5</mu1>
-      <mu2>0.2</mu2>
-      <fdir1>.5 0 0</fdir1>
-      <maxVel>3.0</maxVel>
-      <minDepth>0.00</minDepth>
-      <implicitSpringDamper>3</implicitSpringDamper>
+      <kp>1000000.0</kp>
+      <kd>100.0</kd>
+	  <mu1>0.0</mu1>
+	  <mu2>0.0</mu2>
+	  <minDepth>0.0001</minDepth>
+	  <maxVel>1.0</maxVel>
 </gazebo>
   </xacro:macro>

File: cme_description/robots/mm_400/urdf/xacros/mp_400_gazebo.xacro (robot description, xacro)
@@ -1,16 +1,16 @@
 <?xml version="1.0"?>
 <robot name="mm_400" xmlns:xacro="http://www.ros.org/wiki/xacro">
-   <gazebo reference="base_link">
-    <gravity>true</gravity>
-    <self_collide>false</self_collide>
-  </gazebo>
-  <gazebo reference="castor_wheel_link">
-    <gravity>true</gravity>
-    <self_collide>false</self_collide>
-  </gazebo>
-  <gazebo reference="fixed_wheel_link">
-    <gravity>true</gravity>
-    <self_collide>false</self_collide>
-  </gazebo>
+	<gazebo reference="base_link">
+		<gravity>true</gravity>
+		<self_collide>false</self_collide>
+	</gazebo>
+	<gazebo reference="castor_wheel_link">
+		<gravity>true</gravity>
+		<self_collide>false</self_collide>
+	</gazebo>
+	<gazebo reference="wheel_link">
+		<gravity>true</gravity>
+		<self_collide>false</self_collide>
+	</gazebo>
   <gazebo reference="lidar_1_link">
       <sensor type="ray" name="lidar_1_link">
@@ -48,32 +48,8 @@
         </sensor>
   </gazebo>
-  <gazebo>
-    <plugin name="diff_dirve_controller" filename="libgazebo_ros_diff_drive.so">
-        <alwaysOn>true</alwaysOn>
-        <updateRate>40</updateRate>
-        <legacyMode>false</legacyMode>
-        <torque>0.05</torque>
-        <leftJoint>fixed_wheel_left_joint</leftJoint>
-        <rightJoint>fixed_wheel_right_joint</rightJoint>
-        <wheelSeparation>0.529</wheelSeparation>
-        <wheelDiameter>0.15</wheelDiameter>
-        <commandTopic>cmd_vel</commandTopic>
-        <rosDebugLevel>na</rosDebugLevel>
-        <odometryTopic>odom</odometryTopic>
-        <odometryFrame>odom</odometryFrame>
-        <robotBaseFrame>base_link</robotBaseFrame>
-        <publishWheelTF>true</publishWheelTF>
-        <publishWheelJointState>true</publishWheelJointState>
-        <wheelAcceleration>6.0</wheelAcceleration>
-        <wheelTorque>200</wheelTorque>
-        <odometrySource>world</odometrySource>
-        <publishTf>1</publishTf>
-        <publishOdomTF>true</publishOdomTF>
-    </plugin>
-  </gazebo>
 <gazebo>
   <plugin name="ros_control" filename="libgazebo_ros_control.so">
     <robotNamespace>$(arg robot_namespace)</robotNamespace>
-    <legacyModeNS>false</legacyModeNS>
+    <legacyModeNS>true</legacyModeNS>
     <robotSimType>gazebo_ros_control/DefaultRobotHWSim</robotSimType>
   </plugin>

Commit message: Various controller and manipulator reorg

File: cme_description/robots/mm_400/mm_400.urdf.xacro (robot description, xacro)
@@ -3,5 +3,5 @@
 <robot xmlns:xacro="http://www.ros.org/wiki/xacro" name="mm_400">
 	<xacro:arg name="robot_namespace" default="/" />
-	<xacro:arg name="manipulator" default="pilz" />
+	<xacro:arg name="manipulator" default="" />
 	<xacro:arg name="gripper" default="true" />
 	<xacro:arg name="camera" default="false" />
@@ -18,13 +18,15 @@
 	<xacro:include filename="$(find cme_description)/robots/mm_400/urdf/xacros/mp_400_body.xacro" />
 	<xacro:include filename="$(find cme_description)/robots/mm_400/urdf/xacros/mp_400_caster_wheel.xacro" />
-	<xacro:include filename="$(find cme_description)/robots/mm_400/urdf/xacros/mp_400_wheel_left.xacro" />
-	<xacro:include filename="$(find cme_description)/robots/mm_400/urdf/xacros/mp_400_wheel_right.xacro" />
+	<xacro:include filename="$(find cme_description)/robots/mm_400/urdf/xacros/mp_400_wheel.xacro" />
 	<xacro:include filename="$(find cme_description)/robots/mm_400/urdf/xacros/cabinet.xacro" />
 	<!-- manipulators -->
 	<xacro:if value="$(eval manipulator == 'pilz')">
-		<xacro:include filename="$(find prbt_support)/urdf/prbt_macro.xacro" />
+		<xacro:include filename="$(find prbt_support)/urdf/prbt_macro.xacro"/>
 	</xacro:if>
 	<xacro:if value="$(eval manipulator == 'panda')">
-		<xacro:include filename="$(find franka_description)/robots/panda_arm.xacro" />
+		<xacro:include filename="$(find franka_description)/robots/panda_arm.xacro"/>
+		<xacro:if value="$(arg gripper)">
+			<xacro:include filename="$(find franka_description)/robots/hand.xacro"/>
+		</xacro:if>
 	</xacro:if>
 	<!-- SENSORS -->
@@ -60,8 +62,8 @@
 		<origin xyz="-0.220 -0.155 0.036" rpy="0 0 1.57" />
 	</xacro:caster_wheel>
-	<xacro:wheel name="wheel_right" parent="base_link">
+	<xacro:wheel name="right" parent="base_link">
 		<origin xyz="0. -0.26 0.074" rpy="0 0 1.57" />
 	</xacro:wheel>
-	<xacro:wheel name="wheel_left" parent="base_link">
+	<xacro:wheel name="left" parent="base_link">
 		<origin xyz="-0. 0.26 0.074" rpy="0 0 1.57" />
 	</xacro:wheel>
@@ -73,16 +75,15 @@
 	-->
 	<!-- Robot arm -->
-	<xacro:if value="${eval manipulator == 'pilz'}">
-		<xacro:prbt parent="base_link" prefix="pilz">
-			<origin xyz="0 0 0." rpy="0 0 0" />
-			<xacro:arg name="gripper" value="$(arg gripper)"/>
-		</xacro:prbt>
+	<xacro:if value="$(eval manipulator == 'pilz')">
+		<xacro:prbt prefix="pilz"/>
+		<joint name="pilz-base_link" type="fixed">
+			<parent link="base_link"/>
+			<child link="pilzbase_link"/>
+		</joint>
 	</xacro:if>
 	<!-- Panda -->
-	<xacro:if value="${eval manipulator == 'panda'}">
-		<xacro:panda_arm parent="base_link" prefix="panda">
-			<origin xyz="0 0 0." rpy="0 0 0" />
-			<xacro:arg name="gripper" value="$(arg gripper)"/>
-		</xacro:panda_arm>
+	<xacro:if value="$(eval manipulator == 'panda')">
+		<xacro:panda_arm connected_to="cabinet_link"/>
+		<xacro:hand ns="panda" rpy="0 0 ${-pi/4}" connected_to="panda_link8"/>
 	</xacro:if>
 	<!--

File: cme_description/robots/mm_400/urdf/xacros/mp_400_wheel.xacro (robot description, xacro)
@@ -6,9 +6,9 @@
 				<mass value="2" />
 				<origin xyz="0 0 0" />
-				<inertia ixxx="0.2467" ixy="0" ixz="0"
+				<inertia ixx="0.2467" ixy="0" ixz="0"
 				         iyy="0.04411" iyz="0" izz="0.02467" />
 			</inertial>
 			<visual>
-				<origin xyz="0 0 0" rpy="0 0 0">
+				<origin xyz="0 0 0" rpy="0 0 0"/>
 				<geometry>
 					<mesh filename="package://neo_simulation/robots/mp_400/meshes/MP-400-FIXED-WHEEL-LEFT.dae" scale="0.001 0.001 0.001"/>
@@ -24,5 +24,5 @@
 		<gazebo reference="${name}_wheel_link">
 			<mu1 value="1.0"/>
-			<mu2 value="!.0"/>
+			<mu2 value="1.0"/>
 			<kp value="100000.0" />
 			<kd value="1.0" />

File: cme_description/urdf/complete_model.urdf.xacro (robot description, xacro)
@@ -5,4 +5,5 @@
 	-->
 	<xacro:arg name="world_namespace" default="/" />
+	<xacro:arg name="building" default="mp_model" />
 	<!--
 	 Includes
@@ -18,5 +19,5 @@
 	 Building
 	-->
-	<xacro:include filename="$(find cme_description)/urdf/mp_model.urdf.xacro" />
+	<xacro:include filename="$(find cme_description)/urdf/$(arg building).urdf.xacro" />
 	<!--
 	 Doors
