Commit message: Update mm_400, fix gazebo world

File: cme_description/robots/mm_400/mm_400.urdf.xacro (robot description, xacro)
@@ -7,5 +7,5 @@
 	<xacro:arg name="camera" default="false" />
 	<xacro:arg name="micro_scan" default="true" />
-	<xacro:arg name="sick_S300" default="false" />
+	<xacro:arg name="sick_S300" default="true" />
 	<xacro:arg name="imu" default="false" />
 	<xacro:arg name="ultrasonic" default="false" />
@@ -50,4 +50,10 @@
 	-->
 	<xacro:mp_400_base name="base_link"/>
+	<link name="base_footprint"/>
+	<joint name="base_footprint_joint" type="fixed">
+		<origin xyz="0 0 0" rpy="0 0 0" />
+		<parent link="base_link" />
+		<child link="base_footprint" />
+	</joint>
 	<xacro:caster_wheel name="wheel_front_left" parent="base_link">
 		<origin xyz="0.165 0.155 0.036" rpy="0 0 1.57" />

File: cme_description/robots/mm_400/urdf/xacros/cabinet.xacro (robot description, xacro)
@@ -1,32 +1,32 @@
 <?xml version="1.0"?>
 <robot xmlns:xacro="http://www.ros.org/wiki/xacro" name="mm_400">
-  <xacro:macro name="mm_400_cabinet" params="name parent *origin">
-   <joint name="${name}_joint" type="fixed">
-   <xacro:insert_block name="origin" />
-    <joint_properties damping="1" friction="1" />
-    <parent link="${parent}" />
-    <child link="${name}_link" />
-   </joint>
-    <link name="${name}_link">
-      <inertial>
-        <mass value="1" />
-        <origin xyz="0 0 0" rpy="0 0 0"/>
-        <inertia ixx="1.71402" ixy="0.0" ixz="0.0"
-                 iyy="0.8856" iyz="0.0"
-                 izz="2.5725" />
-      </inertial>
-      <visual>
-        <origin xyz="0 0 0" rpy="0 0 -1.5708" />
-        <geometry>
-            <mesh filename="package://neo_simulation/robots/mm_400/meshes/top.dae" scale="0.001 0.001 0.001"/>
-        </geometry>
-      </visual>
-      <collision>
-        <origin xyz="0. 0. 0" rpy="0 0 0" />
-        <geometry>
-            <mesh filename="package://neo_simulation/robots/mm_400/meshes/top.dae" scale="0.001 0.001 0.001"/>
-        </geometry>
-      </collision>
-    </link>
-  </xacro:macro>
+	<xacro:macro name="mm_400_cabinet" params="name parent *origin">
+	 <joint name="${name}_joint" type="fixed">
+	 <xacro:insert_block name="origin" />
+		<joint_properties damping="1" friction="1" />
+		<parent link="${parent}" />
+		<child link="${name}_link" />
+	 </joint>
+		<link name="${name}_link">
+			<inertial>
+				<mass value="1" />
+				<origin xyz="0 0 0" rpy="0 0 0"/>
+				<inertia ixx="1.71402" ixy="0.0" ixz="0.0"
+								 iyy="0.8856" iyz="0.0"
+								 izz="2.5725" />
+			</inertial>
+			<visual>
+			<origin xyz="0 0 0" rpy="0 0 -${pi/2}" />
+				<geometry>
+						<mesh filename="package://neo_simulation/robots/mm_400/meshes/top.dae" scale="0.001 0.001 0.001"/>
+				</geometry>
+			</visual>
+			<collision>
+				<origin xyz="0. 0. 0" rpy="0 0 -${pi/2}" />
+				<geometry>
+						<mesh filename="package://neo_simulation/robots/mm_400/meshes/top.dae" scale="0.001 0.001 0.001"/>
+				</geometry>
+			</collision>
+		</link>
+	</xacro:macro>
 </robot>

File: cme_description/robots/mm_400/urdf/xacros/mp_400_body.xacro (robot description, xacro)
@@ -1,29 +1,28 @@
 <?xml version="1.0"?>
 <robot xmlns:xacro="http://www.ros.org/wiki/xacro" name="mp_400">
-  <xacro:macro name="mp_400_base" params="name">
-    <link name="${name}">
-  <inertial>
-        <mass value="30" />
-        <origin xyz="0 0 0" rpy="0 0 0"/>
-        <inertia ixx="1.71402" ixy="0.0" ixz="0.0"
-                 iyy="0.8856" iyz="0.0"
-                 izz="2.5725" />
-</inertial>
-      <visual name='body'>
-      <origin xyz="0.0 0.0 0." rpy="0 0 1.57" />
-        <geometry>
-            <mesh filename="package://neo_simulation/robots/mp_400/meshes/MP-400-BODY.dae" scale="0.001 0.001 0.001"/>
-        <!--cylinder length="0.381" radius="0.2545"/-->
-        <!--box size="0.445 0.277 0.17"/-->
-        </geometry>
-      </visual>
-      <collision name='body_collision'>
-        <origin xyz="0.0 0.0 0.0" rpy="0 0 1.57" />
-        <geometry>
-          <mesh filename="package://neo_simulation/robots/mp_400/meshes/MP-400-BODY.dae" scale="0.001 0.001 0.001"/>
-          <!--cylinder length="0.381" radius="0.2545"/-->
-        </geometry>
-      </collision>
-    </link>
-  </xacro:macro>
+	<xacro:macro name="mp_400_base" params="name">
+		<link name="${name}">
+			<inertial>
+				<mass value="30" />
+				<origin xyz="0 0 0" rpy="0 0 0"/>
+				<inertia ixx="1.71402" ixy="0.0" ixz="0.0"
+				         iyy="0.8856" iyz="0.0" izz="2.5725" />
+			</inertial>
+			<visual name='body'>
+			<origin xyz="0.0 0.0 0.0" rpy="0 0 ${pi/2}" />
+				<geometry>
+					<mesh filename="package://neo_simulation/robots/mp_400/meshes/MP-400-BODY.dae" scale="0.001 0.001 0.001"/>
+				<!--cylinder length="0.381" radius="0.2545"/-->
+				<!--box size="0.445 0.277 0.17"/-->
+				</geometry>
+			</visual>
+			<collision name='body_collision'>
+				<origin xyz="0.0 0.0 0.0" rpy="0 0 ${pi/2}" />
+				<geometry>
+					<mesh filename="package://neo_simulation/robots/mp_400/meshes/MP-400-BODY.dae" scale="0.001 0.001 0.001"/>
+					<!--cylinder length="0.381" radius="0.2545"/-->
+				</geometry>
+			</collision>
+		</link>
+	</xacro:macro>
 </robot>

File: cme_description/robots/mm_400/urdf/xacros/mp_400_wheel.xacro (robot description, xacro)
@@ -1,5 +1,5 @@
 <?xml version="1.0"?>
 <robot xmlns:xacro="http://www.ros.org/wiki/xacro" name="mp_400_wheel">
-	<xacro:macro name="wheel" params="name parent *joint_origin wheel_length:=0.2 wheel_radius=0.079">
+	<xacro:macro name="wheel" params="name parent *joint_origin wheel_length:=0.025 wheel_radius=0.079">
 		<link name="${name}_wheel_link">
 			<inertial>
@@ -16,5 +16,5 @@
 			</visual>
 			<collision>
-				<origin xyz="0 0 0" rpy="${pi/2} 0 0" />
+				<origin xyz="0 0 0" rpy="0 ${pi/2} 0" />
 				<geometry>
 					<cylinder length="${wheel_length}" radius="${wheel_radius}" />
@@ -33,5 +33,5 @@
 			<child link="${name}_wheel_link"/>
 			<xacro:insert_block name="joint_origin"/>
-			<axis xyz="0 1 0" rpy="0 0 0"/>
+			<axis xyz="1 0 0" rpy="0 0 0"/>
 		</joint>
 		<transmission name="${name}_wheel_trans" type="SimpleTransmission">

File: cme_description/robots/panda.urdf.xacro (robot description, xacro)
@@ -23,7 +23,7 @@
 	<xacro:panda_arm/>
 	<!-- Override panda connect_to arg -->
-	<xacro:if value="$(eval parent != '')">
-		<joint name="panda_joint_$(arg parent)" type="fixed">
-			<parent link="$(arg parent)"/>
+	<xacro:if value="${parent != ''}">
+		<joint name="panda_joint_${parent}" type="fixed">
+			<parent link="${parent}"/>
 			<child link="panda_link0"/>
 			<origin rpy="$(arg rpy)" xyz="$(arg xyz)"/>
