Commit message: Attempts at fixing mm400

File: cme_description/robots/mm_400/mm_400.urdf.xacro (robot description, xacro)
@@ -7,6 +7,6 @@
 	<xacro:arg name="camera" default="false" />
 	<xacro:arg name="micro_scan" default="true" />
-	<xacro:arg name="sick_S300" default="true" />
-	<xacro:arg name="imu" default="false" />
+	<xacro:arg name="sick_S300" default="false" />
+	<xacro:arg name="imu" default="true" />
 	<xacro:arg name="ultrasonic" default="false" />
 	<xacro:property name="robot_namespace" value="$(arg robot_namespace)"/>
@@ -31,7 +31,8 @@
 	</xacro:if>
 	<!-- SENSORS -->
-	<xacro:if value="$(arg sick_S300)">
+	<!-- TODO: The sick S300 urdf is not complete... -->
+	<!--xacro:if value="$(arg sick_S300)">
 		<xacro:include filename="$(find cme_description)/robots/mm_400/urdf/xacros/sick_S300.xacro" />
-	</xacro:if>
+	</xacro:if-->
 	<xacro:if value="$(arg micro_scan)">
 		<xacro:include filename="$(find cme_description)/robots/mm_400/urdf/xacros/micro_scan.xacro" />
@@ -57,23 +58,23 @@
 	</joint>
 	<xacro:caster_wheel name="wheel_front_left" parent="base_link">
-		<origin xyz="0.165 0.155 0.036" rpy="0 0 1.57" />
+		<origin xyz="0.165 0.155 0.036" rpy="0 0 ${pi/2}" />
 	</xacro:caster_wheel>
 	<xacro:caster_wheel name="wheel_back_left" parent="base_link">
-		<origin xyz="-0.220 0.155 0.036" rpy="0 0 1.57" />
+		<origin xyz="-0.220 0.155 0.036" rpy="0 0 ${pi/2}" />
 	</xacro:caster_wheel>
 	<xacro:caster_wheel name="wheel_front_right" parent="base_link">
-		<origin xyz="0.165 -0.155 0.036" rpy="0 0 1.57" />
+		<origin xyz="0.165 -0.155 0.036" rpy="0 0 ${pi/2}" />
 	</xacro:caster_wheel>
 	<xacro:caster_wheel name="wheel_back_right" parent="base_link">
-		<origin xyz="-0.220 -0.155 0.036" rpy="0 0 1.57" />
+		<origin xyz="-0.220 -0.155 0.036" rpy="0 0 ${pi/2}" />
 	</xacro:caster_wheel>
 	<xacro:wheel name="right" parent="base_link">
-		<origin xyz="0. -0.26 0.074" rpy="0 0 1.57" />
+		<origin xyz="0. -0.26 0.074" rpy="0 0 ${pi/2}" />
 	</xacro:wheel>
 	<xacro:wheel name="left" parent="base_link">
-		<origin xyz="-0. 0.26 0.074" rpy="0 0 1.57" />
+		<origin xyz="-0. 0.26 0.074" rpy="0 0 ${pi/2}" />
 	</xacro:wheel>
 	<xacro:mm_400_cabinet name="cabinet" parent="base_link">
-		<origin xyz="0.02 0 0.551" rpy="0 0 3.14" />
+		<origin xyz="0.02 0 0.551" rpy="0 0 ${pi}" />
 	</xacro:mm_400_cabinet>
 	<!--
@@ -97,6 +98,6 @@
 	-->
 	<xacro:if value="$(arg micro_scan)">
-		<xacro:sick_laser_v0 name="lidar_1" parent="base_link" ros_topic="lidar_1/scan_filtered">
-			<origin xyz="0.230 0 0.110" rpy="0 3.14 3.14" />
+		<xacro:sick_laser_v0 name="lidar_1" parent="base_link" ros_topic="scan">
+			<origin xyz="0.230 0 0.110" rpy="0 ${pi} ${pi}" />
 		</xacro:sick_laser_v0>
 	</xacro:if>
@@ -108,70 +109,70 @@
 	<xacro:if value="$(arg imu)">
 		<xacro:imu name="imu_1" parent="base_link">
-			<origin xyz="0.100 0 0.300" rpy="0 0 3.14" />
+			<origin xyz="0.100 0 0.300" rpy="0 0 ${pi}" />
 		</xacro:imu>
 	</xacro:if>
 	<xacro:if value="$(arg ultrasonic)">
 		<xacro:us_sensor name="us_1" parent="base_link">
-			<origin xyz="0.100 0 0.300" rpy="0 3.14 3.14" />
+			<origin xyz="0.100 0 0.300" rpy="0 ${pi} ${pi}" />
 		</xacro:us_sensor>
 		<!-- SENSOR 2 -->
 		<xacro:us_sensor name="us_2" parent="base_link">
-			<origin xyz="0.110 0 0.300" rpy="0 3.14 3.14" />
+			<origin xyz="0.110 0 0.300" rpy="0 ${pi} ${pi}" />
 		</xacro:us_sensor>
 		<!-- SENSOR 3 -->
 		<xacro:us_sensor name="us_3" parent="base_link">
-			<origin xyz="0.120 0 0.300" rpy="0 3.14 3.14" />
+			<origin xyz="0.120 0 0.300" rpy="0 ${pi} ${pi}" />
 		</xacro:us_sensor>
 		<!-- SENSOR 4 -->
 		<xacro:us_sensor name="us_4" parent="base_link">
-			<origin xyz="0.130 0 0.300" rpy="0 3.14 3.14" />
+			<origin xyz="0.130 0 0.300" rpy="0 ${pi} ${pi}" />
 		</xacro:us_sensor>
 		<!-- SENSOR 5 -->
 		<xacro:us_sensor name="us_5" parent="base_link">
-			<origin xyz="0.140 0 0.300" rpy="0 3.14 3.14" />
+			<origin xyz="0.140 0 0.300" rpy="0 ${pi} ${pi}" />
 		</xacro:us_sensor>
 		<!-- SENSOR 6 -->
 		<xacro:us_sensor name="us_6" parent="base_link">
-			<origin xyz="0.150 0 0.300" rpy="0 3.14 3.14" />
+			<origin xyz="0.150 0 0.300" rpy="0 ${pi} ${pi}" />
 		</xacro:us_sensor>
 		<!-- SENSOR 7 -->
 		<xacro:us_sensor name="us_7" parent="base_link">
-			<origin xyz="0.160 0 0.300" rpy="0 3.14 3.14" />
+			<origin xyz="0.160 0 0.300" rpy="0 ${pi} ${pi}" />
 		</xacro:us_sensor>
 		<!-- SENSOR 8 -->
 		<xacro:us_sensor name="us_8" parent="base_link">
-			<origin xyz="0.170 0 0.300" rpy="0 3.14 3.14" />
+			<origin xyz="0.170 0 0.300" rpy="0 ${pi} ${pi}" />
 		</xacro:us_sensor>
 		<!-- SENSOR 9 -->
 		<xacro:us_sensor name="us_9" parent="base_link">
-			<origin xyz="0.180 0 0.300" rpy="0 3.14 3.14" />
+			<origin xyz="0.180 0 0.300" rpy="0 ${pi} ${pi}" />
 		</xacro:us_sensor>
 		<!-- SENSOR 10 -->
 		<xacro:us_sensor name="us_10" parent="base_link">
-			<origin xyz="0.100 0 0.300" rpy="0 3.14 3.14" />
+			<origin xyz="0.100 0 0.300" rpy="0 ${pi} ${pi}" />
 		</xacro:us_sensor>
 		<!-- SENSOR 11 -->
 		<xacro:us_sensor name="us_11" parent="base_link">
-			<origin xyz="0.100 0 0.300" rpy="0 3.14 3.14" />
+			<origin xyz="0.100 0 0.300" rpy="0 ${pi} ${pi}" />
 		</xacro:us_sensor>
 		<!-- SENSOR 12 -->
 		<xacro:us_sensor name="us_12" parent="base_link">
-			<origin xyz="0.190 0 0.300" rpy="0 3.14 3.14" />
+			<origin xyz="0.190 0 0.300" rpy="0 ${pi} ${pi}" />
 		</xacro:us_sensor>
 		<!-- SENSOR 13 -->
 		<xacro:us_sensor name="us_13" parent="base_link">
-			<origin xyz="0.200 0 0.300" rpy="0 3.14 3.14" />
+			<origin xyz="0.200 0 0.300" rpy="0 ${pi} ${pi}" />
 		</xacro:us_sensor>
 		<!-- SENSOR 14 -->
 		<xacro:us_sensor name="us_14" parent="base_link">
-			<origin xyz="0.210 0 0.300" rpy="0 3.14 3.14" />
+			<origin xyz="0.210 0 0.300" rpy="0 ${pi} ${pi}" />
 		</xacro:us_sensor>
 		<!-- SENSOR 15 -->
 		<xacro:us_sensor name="us_15" parent="base_link">
-			<origin xyz="0.220 0 0.300" rpy="0 3.14 3.14" />
+			<origin xyz="0.220 0 0.300" rpy="0 ${pi} ${pi}" />
 		</xacro:us_sensor>
 		<!-- SENSOR 16 -->
 		<xacro:us_sensor name="us_16" parent="base_link">
-			<origin xyz="0.230 0 0.300" rpy="0 3.14 3.14" />
+			<origin xyz="0.230 0 0.300" rpy="0 ${pi} ${pi}" />
 		</xacro:us_sensor>
 	</xacro:if>

File: cme_description/robots/mm_400/urdf/xacros/cabinet.xacro (robot description, xacro)
@@ -2,10 +2,9 @@
 <robot xmlns:xacro="http://www.ros.org/wiki/xacro" name="mm_400">
 	<xacro:macro name="mm_400_cabinet" params="name parent *origin">
-	 <joint name="${name}_joint" type="fixed">
-	 <xacro:insert_block name="origin" />
-		<joint_properties damping="1" friction="1" />
-		<parent link="${parent}" />
-		<child link="${name}_link" />
-	 </joint>
+		<joint name="${name}_joint" type="fixed">
+			<xacro:insert_block name="origin" />
+			<parent link="${parent}" />
+			<child link="${name}_link" />
+		</joint>
 		<link name="${name}_link">
 			<inertial>
@@ -17,5 +16,5 @@
 			</inertial>
 			<visual>
-			<origin xyz="0 0 0" rpy="0 0 -${pi/2}" />
+				<origin xyz="0 0 0" rpy="0 0 -${pi/2}" />
 				<geometry>
 						<mesh filename="package://neo_simulation/robots/mm_400/meshes/top.dae" scale="0.001 0.001 0.001"/>
@@ -23,5 +22,5 @@
 			</visual>
 			<collision>
-				<origin xyz="0. 0. 0" rpy="0 0 -${pi/2}" />
+				<origin xyz="0 0 0" rpy="0 0 -${pi/2}" />
 				<geometry>
 						<mesh filename="package://neo_simulation/robots/mm_400/meshes/top.dae" scale="0.001 0.001 0.001"/>

File: cme_description/robots/mm_400/urdf/xacros/micro_scan.xacro (robot description, xacro)
@@ -15,5 +15,5 @@
       </inertial>
       <visual>
-        <origin xyz="-0.0 0 -0.06" rpy="1.57 0 0" />
+        <origin xyz="-0.0 0 -0.06" rpy="${pi/2} 0 0" />
         <geometry>
         <mesh filename="package://neo_simulation/robots/mm_400/meshes/SICK-MICROSCAN3.dae" scale="0.001 0.001 0.001" />
@@ -21,5 +21,5 @@
       </visual>
       <collision>
-        <origin xyz="-0.0 0 -0.06" rpy="1.57 0 0" />
+        <origin xyz="-0.0 0 -0.06" rpy="${pi/2} 0 0" />
         <geometry>
         <mesh filename="package://neo_simulation/robots/mm_400/meshes/SICK-MICROSCAN3.dae" scale="0.001 0.001 0.001" />

File: cme_description/robots/mm_400/urdf/xacros/mp_400_caster_wheel.xacro (robot description, xacro)
@@ -1,41 +1,41 @@
 <?xml version="1.0"?>
 <robot xmlns:xacro="http://www.ros.org/wiki/xacro" name="mp_400">
-  <xacro:macro name="caster_wheel" params="name parent *origin">
-   <joint name="${name}_joint" type="fixed">
-    <xacro:insert_block name="origin" />
-    <axis xyz="-1 0 0" />
-    <joint_properties damping="1" friction="1" />
-    <limit effort="1000.0" lower="-1e+16" upper="1e+16" velocity="3.5"/>
-    <parent link="${parent}" />
-    <child link="${name}_link" />
-   </joint>
-   <link name="${name}_link" type="wheel">
-   <inertial>
-        <mass value="1.4"/>
-        <inertia ixx="0.00499743171" ixy="0.0" ixz="-0.0"
-                 iyy="0.00499741733" iyz="-0.0"
-                 izz="0.00839239692"/>
-  </inertial>
-      <visual name='caster_wheel'>
-    <origin xyz="0 0 0" rpy="0 0 0" />
-    <geometry>
-            <mesh filename="package://neo_simulation/robots/mp_400/meshes/MP-400-CASTER-WHEEL.dae" scale="0.001 0.001 0.001"/>
-    </geometry>
-    </visual>
-    <collision>
-      <origin xyz="0 0. 0" rpy="0 0 0" />
-      <geometry>
-          <sphere radius="0.040"/>
-      </geometry>
-    </collision>
-    </link>
-<gazebo reference="${name}_link">
-      <kp>1000000.0</kp>
-      <kd>100.0</kd>
-	  <mu1>0.0</mu1>
-	  <mu2>0.0</mu2>
-	  <minDepth>0.0001</minDepth>
-	  <maxVel>1.0</maxVel>
-</gazebo>
-  </xacro:macro>
+	<xacro:macro name="caster_wheel" params="name parent *origin">
+		<joint name="${name}_joint" type="fixed">
+			<xacro:insert_block name="origin" />
+			<axis xyz="-1 0 0" />
+			<joint_properties damping="1" friction="1" />
+			<dynamics damping="1" friction="1"/>
+			<limit effort="1000.0" lower="-1e+16" upper="1e+16" velocity="3.5"/>
+			<parent link="${parent}" />
+			<child link="${name}_link" />
+		</joint>
+		<link name="${name}_link" type="wheel">
+			<inertial>
+				<mass value="1.4"/>
+				<inertia ixx="0.00499743171" ixy="0.0" ixz="-0.0"
+						iyy="0.00499741733" iyz="-0.0" izz="0.00839239692"/>
+			</inertial>
+			<visual name='caster_wheel'>
+				<origin xyz="0 0 0" rpy="0 0 0" />
+				<geometry>
+					<mesh filename="package://neo_simulation/robots/mp_400/meshes/MP-400-CASTER-WHEEL.dae" scale="0.001 0.001 0.001"/>
+				</geometry>
+			</visual>
+			<collision>
+				<origin xyz="0 0. 0" rpy="0 0 0" />
+				<geometry>
+					<sphere radius="0.040"/>
+				</geometry>
+			</collision>
+		</link>
+		<gazebo reference="${name}_link">
+			<kp>1000000.0</kp>
+			<kd>100.0</kd>
+			<mu1>0.0</mu1>
+			<mu2>0.0</mu2>
+			<minDepth>0.001</minDepth>
+			<maxVel>1.0</maxVel>
+		</gazebo>
+	</xacro:macro>
 </robot>

File: cme_description/robots/mm_400/urdf/xacros/mp_400_gazebo.xacro (robot description, xacro)
@@ -13,139 +13,141 @@
 		<self_collide>false</self_collide>
 	</gazebo>
-  <gazebo reference="lidar_1_link">
-      <sensor type="ray" name="lidar_1_link">
-          <pose>0 0 0 0 0 0</pose>
-          <visualize>false</visualize>
-          <update_rate>40</update_rate>
-          <ray>
-            <scan>
-              <horizontal>
-                <samples>720</samples>
-                <resolution>1</resolution>
-                <min_angle>-0.785398</min_angle>
-                <max_angle>0.785398</max_angle>
-              </horizontal>
-            </scan>
-            <range>
-              <min>0.10</min>
-              <max>30.0</max>
-              <resolution>0.05</resolution>
-            </range>
-            <noise>
-              <type>gaussian</type>
-              <!-- Noise parameters based on published spec for Hokuyo laser
-                   achieving "+-30mm" accuracy at range < 10m.  A mean of 0.0m and
-                   stddev of 0.01m will put 99.7% of samples within 0.03m of the true
-                   reading. -->
-              <mean>0.0</mean>
-              <stddev>0.01</stddev>
-            </noise>
-          </ray>
-          <plugin name="lidar_1_link" filename="libgazebo_ros_laser.so">
-            <topicName>lidar_1/scan_filtered</topicName>
-            <frameName>lidar_1_link</frameName>
-          </plugin>
-        </sensor>
-  </gazebo>
-<gazebo>
-  <plugin name="ros_control" filename="libgazebo_ros_control.so">
-    <robotNamespace>$(arg robot_namespace)</robotNamespace>
-    <legacyModeNS>true</legacyModeNS>
-    <robotSimType>gazebo_ros_control/DefaultRobotHWSim</robotSimType>
-  </plugin>
-</gazebo>
-  <gazebo reference="us_1_link">
-  <!-- Visuals / Collisions omitted for this example -->
-  <sensor type="ray" name="range">
-    <ray>
-         <scan>
-            <horizontal>
-               <samples>1</samples>
-               <resolution>1.0</resolution>
-               <min_angle>-0.01</min_angle>
-               <max_angle>0.01</max_angle>
-            </horizontal>
-            <vertical>
-               <samples>1</samples>
-               <resolution>1</resolution>
-               <min_angle>-0.01</min_angle>
-               <max_angle>0.01</max_angle>
-            </vertical>
-         </scan>
-         <range>
-            <min>0.01</min>
-            <max>3.75</max>
-            <resolution>0.02</resolution>
-         </range>
-      </ray>
-    <plugin name="libgazebo_ros_range" filename="libgazebo_ros_range.so">
-         <gaussianNoise>0.005</gaussianNoise>
-         <alwaysOn>true</alwaysOn>
-         <updateRate>50</updateRate>
-         <topicName>us_sensor</topicName>
-         <frameName>us_1_link</frameName>
-         <radiation>SONAR</radiation>
-         <fov>0.2967</fov>
-    </plugin>
-  </sensor>
-  </gazebo>
-    <!-- camera -->
-  <gazebo reference="camera_link">
-    <sensor type="camera" name="camera1">
-      <update_rate>30.0</update_rate>
-      <camera name="head">
-        <horizontal_fov>1.3962634</horizontal_fov>
-        <image>
-          <width>800</width>
-          <height>800</height>
-          <format>R8G8B8</format>
-        </image>
-        <clip>
-          <near>0.02</near>
-          <far>300</far>
-        </clip>
-        <noise>
-          <type>gaussian</type>
-          <!-- Noise is sampled independently per pixel on each frame.
-               That pixel's noise value is added to each of its color
-               channels, which at that point lie in the range [0,1]. -->
-          <mean>0.0</mean>
-          <stddev>0.007</stddev>
-        </noise>
-      </camera>
-      <plugin name="camera_controller" filename="libgazebo_ros_camera.so">
-        <alwaysOn>true</alwaysOn>
-        <updateRate>0.0</updateRate>
-        <cameraName>camera1</cameraName>
-        <imageTopicName>image_raw</imageTopicName>
-        <cameraInfoTopicName>camera_info</cameraInfoTopicName>
-        <frameName>camera_link</frameName>
-        <hackBaseline>0.07</hackBaseline>
-        <distortionK1>0.0</distortionK1>
-        <distortionK2>0.0</distortionK2>
-        <distortionK3>0.0</distortionK3>
-        <distortionT1>0.0</distortionT1>
-        <distortionT2>0.0</distortionT2>
-      </plugin>
-    </sensor>
-  </gazebo>
-    <gazebo reference="imu_1_link">
-    <gravity>true</gravity>
-    <sensor name="imu_sensor" type="imu">
-      <always_on>true</always_on>
-      <update_rate>100</update_rate>
-      <visualize>true</visualize>
-      <topic>__default_topic__</topic>
-      <plugin filename="libgazebo_ros_imu_sensor.so" name="imu_plugin">
-        <topicName>imu</topicName>
-        <bodyName>imu_link</bodyName>
-        <updateRateHZ>10.0</updateRateHZ>
-        <gaussianNoise>0.0</gaussianNoise>
-        <xyzOffset>0 0 0</xyzOffset>
-        <rpyOffset>0 0 0</rpyOffset>
-        <frameName>imu_link</frameName>
-      </plugin>
-      <pose>0 0 0 0 0 0</pose>
-    </sensor>
-  </gazebo>
+	<gazebo reference="lidar_1_link">
+		<sensor type="ray" name="lidar_1_link">
+			<pose>0 0 0 0 0 0</pose>
+			<visualize>true</visualize>
+			<update_rate>40</update_rate>
+			<ray>
+				<scan>
+					<horizontal>
+						<samples>720</samples>
+						<resolution>1</resolution>
+						<min_angle>-0.785398</min_angle>
+						<max_angle>0.785398</max_angle>
+					</horizontal>
+				</scan>
+				<range>
+					<min>0.10</min>
+					<max>30.0</max>
+					<resolution>0.01</resolution>
+				</range>
+				<noise>
+					<type>gaussian</type>
+					<!-- Noise parameters based on published spec for Hokuyo laser
+								achieving "+-30mm" accuracy at range < 10m.	A mean of 0.0m and
+								stddev of 0.01m will put 99.7% of samples within 0.03m of the true
+								reading. -->
+					<mean>0.0</mean>
+					<stddev>0.001</stddev>
+				</noise>
+			</ray>
+			<plugin name="lidar_1_link" filename="libgazebo_ros_laser.so">
+				<topicName>lidar_1/scan</topicName>
+				<frameName>lidar_1_link</frameName>
+				<robotNamespace>${robot_namespace}</robotNamespace>
+			</plugin>
+		</sensor>
+	</gazebo>
+	<gazebo>
+		<plugin name="gazebo_ros_control" filename="libgazebo_ros_control.so">
+			<robotNamespace>$(arg robot_namespace)</robotNamespace>
+			<legacyModeNS>true</legacyModeNS>
+			<!--robotSimType>gazebo_ros_control/DefaultRobotHWSim</robotSimType-->
+		</plugin>
+	</gazebo>
+	<gazebo reference="us_1_link">
+		<!-- Visuals / Collisions omitted for this example -->
+		<sensor type="ray" name="range">
+			<ray>
+				<scan>
+					<horizontal>
+						<samples>1</samples>
+						<resolution>1.0</resolution>
+						<min_angle>-0.01</min_angle>
+						<max_angle>0.01</max_angle>
+					</horizontal>
+					<vertical>
+						<samples>1</samples>
+						<resolution>1</resolution>
+						<min_angle>-0.01</min_angle>
+						<max_angle>0.01</max_angle>
+					</vertical>
+				</scan>
+				<range>
+					<min>0.01</min>
+					<max>3.75</max>
+					<resolution>0.02</resolution>
+				</range>
+			</ray>
+			<plugin name="libgazebo_ros_range" filename="libgazebo_ros_range.so">
+				<gaussianNoise>0.005</gaussianNoise>
+				<alwaysOn>true</alwaysOn>
+				<updateRate>50</updateRate>
+				<topicName>us_sensor</topicName>
+				<frameName>us_1_link</frameName>
+				<radiation>SONAR</radiation>
+				<fov>0.2967</fov>
+			</plugin>
+		</sensor>
+	</gazebo>
+		<!-- camera -->
+	<gazebo reference="camera_link">
+		<sensor type="camera" name="camera1">
+			<update_rate>30.0</update_rate>
+			<camera name="head">
+				<horizontal_fov>1.3962634</horizontal_fov>
+				<image>
+					<width>800</width>
+					<height>800</height>
+					<format>R8G8B8</format>
+				</image>
+				<clip>
+					<near>0.02</near>
+					<far>300</far>
+				</clip>
+				<noise>
+					<type>gaussian</type>
+					<!-- Noise is sampled independently per pixel on each frame.
+							 That pixel's noise value is added to each of its color
+							 channels, which at that point lie in the range [0,1]. -->
+					<mean>0.0</mean>
+					<stddev>0.007</stddev>
+				</noise>
+			</camera>
+			<plugin name="camera_controller" filename="libgazebo_ros_camera.so">
+				<alwaysOn>true</alwaysOn>
+				<updateRate>0.0</updateRate>
+				<cameraName>camera1</cameraName>
+				<imageTopicName>image_raw</imageTopicName>
+				<cameraInfoTopicName>camera_info</cameraInfoTopicName>
+				<frameName>camera_link</frameName>
+				<hackBaseline>0.07</hackBaseline>
+				<distortionK1>0.0</distortionK1>
+				<distortionK2>0.0</distortionK2>
+				<distortionK3>0.0</distortionK3>
+				<distortionT1>0.0</distortionT1>
+				<distortionT2>0.0</distortionT2>
+			</plugin>
+		</sensor>
+	</gazebo>
+	<gazebo reference="imu_1_link">
+		<gravity>true</gravity>
+		<sensor name="imu_sensor" type="imu">
+			<always_on>true</always_on>
+			<update_rate>100</update_rate>
+			<visualize>true</visualize>
+			<topic>__default_topic__</topic>
+			<plugin filename="libgazebo_ros_imu_sensor.so" name="imu_plugin">
+				<robotNamespace>${robot_namespace}</robotNamespace>
+				<topicName>imu/data</topicName>
+				<bodyName>base_link</bodyName>
+				<updateRateHZ>50.0</updateRateHZ>
+				<gaussianNoise>0.0</gaussianNoise>
+				<xyzOffset>0 0 0</xyzOffset>
+				<rpyOffset>0 0 0</rpyOffset>
+				<frameName>imu_link</frameName>
+			</plugin>
+			<pose>0 0 0 0 0 0</pose>
+		</sensor>
+	</gazebo>
 </robot>

File: cme_description/robots/mm_400/urdf/xacros/mp_400_wheel.xacro (robot description, xacro)
@@ -1,5 +1,5 @@
 <?xml version="1.0"?>
 <robot xmlns:xacro="http://www.ros.org/wiki/xacro" name="mp_400_wheel">
-	<xacro:macro name="wheel" params="name parent *joint_origin wheel_length:=0.025 wheel_radius=0.079">
+	<xacro:macro name="wheel" params="name parent *joint_origin wheel_length:=0.025 wheel_radius=0.078">
 		<link name="${name}_wheel_link">
 			<inertial>
@@ -25,6 +25,7 @@
 			<mu1 value="1.0"/>
 			<mu2 value="1.0"/>
-			<kp value="100000.0" />
-			<kd value="1.0" />
+			<kp value="1000000.0" />
+			<kd value="100.0" />
+			<minDepth>0.001</minDepth>
 			<fdir value="1 0 0"/>
 		</gazebo>
@@ -34,4 +35,5 @@
 			<xacro:insert_block name="joint_origin"/>
 			<axis xyz="1 0 0" rpy="0 0 0"/>
+			<dynamics damping="50" friction="1"/>
 		</joint>
 		<transmission name="${name}_wheel_trans" type="SimpleTransmission">
