Commit message: Attempts at fixing mm400

File: cme_description/robots/mm_400/urdf/xacros/sick_S300.xacro (robot description, xacro)
@@ -1,30 +1,30 @@
 <?xml version="1.0"?>
 <robot xmlns:xacro="http://www.ros.org/wiki/xacro" name="mp_400">
-  <xacro:macro name="sick_laser_v0" params="name parent *origin ros_topic">
-    <joint name="${name}_joint" type="fixed">
-      <axis xyz="0 1 0" />
-      <xacro:insert_block name="origin" />
-      <parent link="${parent}"/>
-      <child link="${name}_link"/>
-    </joint>
-    <link name="${name}_link" type="laser">
-      <inertial>
-        <mass value="0.001" />
-        <origin xyz="0 0 0" rpy="0 0 0" />
-        <inertia ixx="0.0001" ixy="0" ixz="0" iyy="0.000001" iyz="0" izz="0.0001" />
-      </inertial>
-      <visual>
-        <origin xyz="0 0 -0.11" rpy="-1.57 0 3.14" />
-        <geometry>
-        <mesh filename="package://neo_simulation/robots/mp_400/meshes/SICK-MICROSCAN3.dae" scale="0.001 0.001 0.001" />
-        </geometry>
-      </visual>
-      <collision>
-        <origin xyz="0 0 -0.11" rpy="-1.57 0 3.14" />
-        <geometry>
-        <mesh filename="package://neo_simulation/robots/mp_400/meshes/SICK-MICROSCAN3.dae" scale="0.001 0.001 0.001" />
-        </geometry>
-      </collision>
-    </link>
-  </xacro:macro>
+	<xacro:macro name="sick_laser_v0" params="name parent *origin ros_topic">
+		<joint name="${name}_joint" type="fixed">
+			<axis xyz="0 1 0" />
+			<xacro:insert_block name="origin" />
+			<parent link="${parent}"/>
+			<child link="${name}_link"/>
+		</joint>
+		<link name="${name}_link" type="laser">
+			<inertial>
+				<mass value="0.001" />
+				<origin xyz="0 0 0" rpy="0 0 0" />
+				<inertia ixx="0.0001" ixy="0" ixz="0" iyy="0.000001" iyz="0" izz="0.0001" />
+			</inertial>
+			<visual>
+				<origin xyz="0 0 -0.11" rpy="-${pi/2} 0 ${pi}" />
+				<geometry>
+				<mesh filename="package://neo_simulation/robots/mp_400/meshes/SICK-MICROSCAN3.dae" scale="0.001 0.001 0.001" />
+				</geometry>
+			</visual>
+			<collision>
+				<origin xyz="0 0 -0.11" rpy="-${pi/2} 0 ${pi}" />
+				<geometry>
+				<mesh filename="package://neo_simulation/robots/mp_400/meshes/SICK-MICROSCAN3.dae" scale="0.001 0.001 0.001" />
+				</geometry>
+			</collision>
+		</link>
+	</xacro:macro>
 </robot>

File: cme_description/urdf/complete_mp_model.urdf.xacro (robot description, xacro)
@@ -5,4 +5,5 @@
 	-->
 	<xacro:arg name="world_namespace" default="/" />
+	<xacro:arg name="doors" default="true" />
 	<!--
 	 Includes
@@ -43,21 +44,23 @@
 	 Doors
 	-->
-	<xacro:door id="1" parent="building_footprint" width="0.70" height="2.43" depth="0.05" mirror="true"
-		xyz="2.06 -3.5 0.01" rpy="0 0 0"/>
-	<!-- Room 2 doesn't have a door -->
-	<xacro:door id="3" parent="building_footprint" width="0.70" height="2.43" depth="0.05" flip="true"
-		xyz="2.54 -4.02 0" rpy="0 0 ${pi/2}"/>
-	<xacro:door id="4" parent="building_footprint" width="0.70" height="2.43" depth="0.05" flip="true"
-		xyz="3 -4.53 0" rpy="0 0 0"/>
-	<xacro:door id="5" parent="building_footprint" width="0.70" height="2.43" depth="0.05" flip="true"
-		xyz="2.5 -7.6 0" rpy="0 0 ${pi/2}"/>
-	<xacro:door id="6" parent="building_footprint" width="0.70" height="2.43" depth="0.05" flip="true"
-		xyz="0.2 -8.45 0" rpy="0 0 ${pi/2}"/>
-	<xacro:door id="7" parent="building_footprint" width="0.70" height="2.43" depth="0.05" flip="true"
-		xyz="-0.55 -8.95 0" rpy="0 0 0"/>
-	<xacro:door id="8" parent="building_footprint" width="0.70" height="2.43" depth="0.05" flip="true"
-		xyz="2.05 -8.95 0" rpy="0 0 0"/>
-	<xacro:door id="9" parent="building_footprint" width="0.70" height="2.43" depth="0.05" flip="true"
-		xyz="2.5 -8.5 0" rpy="0 0 ${pi/2}"/>
+	<xacro:if value="$(arg doors)">
+		<xacro:door id="1" parent="building_footprint" width="0.70" height="2.43" depth="0.05" mirror="true"
+			xyz="2.06 -3.5 0.01" rpy="0 0 0"/>
+		<!-- Room 2 doesn't have a door -->
+		<xacro:door id="3" parent="building_footprint" width="0.70" height="2.43" depth="0.05" flip="true"
+			xyz="2.54 -4.02 0" rpy="0 0 ${pi/2}"/>
+		<xacro:door id="4" parent="building_footprint" width="0.70" height="2.43" depth="0.05" flip="true"
+			xyz="3 -4.53 0" rpy="0 0 0"/>
+		<xacro:door id="5" parent="building_footprint" width="0.70" height="2.43" depth="0.05" flip="true"
+			xyz="2.5 -7.6 0" rpy="0 0 ${pi/2}"/>
+		<xacro:door id="6" parent="building_footprint" width="0.70" height="2.43" depth="0.05" flip="true"
+			xyz="0.2 -8.45 0" rpy="0 0 ${pi/2}"/>
+		<xacro:door id="7" parent="building_footprint" width="0.70" height="2.43" depth="0.05" flip="true"
+			xyz="-0.55 -8.95 0" rpy="0 0 0"/>
+		<xacro:door id="8" parent="building_footprint" width="0.70" height="2.43" depth="0.05" flip="true"
+			xyz="2.05 -8.95 0" rpy="0 0 0"/>
+		<xacro:door id="9" parent="building_footprint" width="0.70" height="2.43" depth="0.05" flip="true"
+			xyz="2.5 -8.5 0" rpy="0 0 ${pi/2}"/>
+	</xacro:if>
 	<!--
 	 light switches

File: cme_description/urdf/complete_mp_model_wider.urdf.xacro (robot description, xacro)
@@ -5,4 +5,5 @@
 	-->
 	<xacro:arg name="world_namespace" default="/" />
+	<xacro:arg name="doors" default="true" />
 	<!--
 	 Includes
@@ -43,21 +44,23 @@
 	 Doors
 	-->
-	<xacro:door id="1" parent="building_footprint" width="1.4" height="2.43" depth="0.05" mirror="true"
-		xyz="1.85 2.539 0" rpy="0 0 0"/>
-	<!-- Room 2 doesn't have a door -->
-	<xacro:door id="3" parent="building_footprint" width="0.85" height="2.43" depth="0.05" flip="true"
-		xyz="2.59 1.97 0" rpy="0 0 ${pi/2}"/>
-	<xacro:door id="4" parent="building_footprint" width="1.0" height="2.43" depth="0.05" flip="true"
-		xyz="3.15 1.46 0" rpy="0 0 0"/>
-	<xacro:door id="5" parent="building_footprint" width="0.70" height="2.43" depth="0.05" flip="true"
-		xyz="2.57 -1.6 0" rpy="0 0 ${pi/2}"/>
-	<xacro:door id="6" parent="building_footprint" width="1.2" height="2.43" depth="0.05" flip="true"
-		xyz="0.16 -2.48 0" rpy="0 0 ${pi/2}"/>
-	<xacro:door id="7" parent="building_footprint" width="1.0" height="2.43" depth="0.05" flip="true"
-		xyz="-0.42 -3.258 0" rpy="0 0 0"/>
-	<xacro:door id="8" parent="building_footprint" width="1.0" height="2.43" depth="0.05" flip="true"
-		xyz="1.92 -3.258 0" rpy="0 0 0"/>
-	<xacro:door id="9" parent="building_footprint" width="1.0" height="2.43" depth="0.05" flip="true"
-		xyz="2.57 -2.66 0" rpy="0 0 ${pi/2}"/>
+	<xacro:if value="$(arg doors)">
+		<xacro:door id="1" parent="building_footprint" width="1.4" height="2.43" depth="0.05" mirror="true"
+			xyz="1.85 2.539 0" rpy="0 0 0"/>
+		<!-- Room 2 doesn't have a door -->
+		<xacro:door id="3" parent="building_footprint" width="0.85" height="2.43" depth="0.05" flip="true"
+			xyz="2.59 1.97 0" rpy="0 0 ${pi/2}"/>
+		<xacro:door id="4" parent="building_footprint" width="1.0" height="2.43" depth="0.05" flip="true"
+			xyz="3.15 1.46 0" rpy="0 0 0"/>
+		<xacro:door id="5" parent="building_footprint" width="0.70" height="2.43" depth="0.05" flip="true"
+			xyz="2.57 -1.6 0" rpy="0 0 ${pi/2}"/>
+		<xacro:door id="6" parent="building_footprint" width="1.2" height="2.43" depth="0.05" flip="true"
+			xyz="0.16 -2.48 0" rpy="0 0 ${pi/2}"/>
+		<xacro:door id="7" parent="building_footprint" width="1.0" height="2.43" depth="0.05" flip="true"
+			xyz="-0.42 -3.258 0" rpy="0 0 0"/>
+		<xacro:door id="8" parent="building_footprint" width="1.0" height="2.43" depth="0.05" flip="true"
+			xyz="1.92 -3.258 0" rpy="0 0 0"/>
+		<xacro:door id="9" parent="building_footprint" width="1.0" height="2.43" depth="0.05" flip="true"
+			xyz="2.57 -2.66 0" rpy="0 0 ${pi/2}"/>
+	</xacro:if>
 	<!--
 	 light switches
